File: centrifuge/inter_board.kicad_sch (KiCad schematic)
At the start: 0 parts

Commit message: Completed majority of schematic, need to add decoupling but otherwise mostly ready
Other:
- title: (none) -> VGA Centrifuge
Changed lines of the file:
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@@
 (kicad_sch (version 20211123) (generator eeschema)
   (paper "A4")
+  (title_block
+    (title "VGA Centrifuge")
+    (rev "R1")
+    (comment 1 "Author: Paolo Celati")
+  )
 )
