File: centrifuge/centrifuge.kicad_pcb (KiCad board)
At the start: 8 copper layers, 3 parts, among them U1 XC7A100T-FTG256, U2 S25FL127SABMFV10, U3 CY7C1370KV33

Commit message: Completed majority of schematic, need to add decoupling but otherwise mostly ready
Parts:
- added C1: 10u, Capacitor_SMD:C_0805_2012Metric_Pad1.18x1.45mm_HandSolder, F.Cu at (234.2, 103.3)
- added C10: 1u, Capacitor_SMD:C_0805_2012Metric_Pad1.18x1.45mm_HandSolder, F.Cu at (264.3, 115.9)
- added C11: 1u, Capacitor_SMD:C_0805_2012Metric_Pad1.18x1.45mm_HandSolder, F.Cu at (273.9, 106.3)
- added C12: 1u, Capacitor_SMD:C_0805_2012Metric_Pad1.18x1.45mm_HandSolder, F.Cu at (264.3, 118.9)
- added C13: 0.1u, Capacitor_SMD:C_0805_2012Metric_Pad1.18x1.45mm_HandSolder, F.Cu at (259.5, 121.9)
- added C14: 0.1u, Capacitor_SMD:C_0805_2012Metric_Pad1.18x1.45mm_HandSolder, F.Cu at (278.8, 106.3)
- added C15: 0.1u, Capacitor_SMD:C_0805_2012Metric_Pad1.18x1.45mm_HandSolder, F.Cu at (259.5, 115.9)
- added C16: 1u, Capacitor_SMD:C_0805_2012Metric_Pad1.18x1.45mm_HandSolder, F.Cu at (259.5, 106.9)
- added C17: 10n, Capacitor_SMD:C_0805_2012Metric_Pad1.18x1.45mm_HandSolder, F.Cu at (264.3, 112.9)
- added C18: 1u, Capacitor_SMD:C_0805_2012Metric_Pad1.18x1.45mm_HandSolder, F.Cu at (283.6, 106.3)
- added C19: 10n, Capacitor_SMD:C_0805_2012Metric_Pad1.18x1.45mm_HandSolder, F.Cu at (273.9, 112.4)
- added C2: 10u, Capacitor_SMD:C_0805_2012Metric_Pad1.18x1.45mm_HandSolder, F.Cu at (229.4, 109.3)
- added C20: 0.1u, Capacitor_SMD:C_0805_2012Metric_Pad1.18x1.45mm_HandSolder, F.Cu at (264.3, 121.9)
- added C21: 10n, Capacitor_SMD:C_0805_2012Metric_Pad1.18x1.45mm_HandSolder, F.Cu at (259.5, 112.9)
- added C22: 10n, Capacitor_SMD:C_0805_2012Metric_Pad1.18x1.45mm_HandSolder, F.Cu at (265.2, 103.3)
- added C23: 1u, Capacitor_SMD:C_0805_2012Metric_Pad1.18x1.45mm_HandSolder, F.Cu at (278.8, 109.3)
- added C24: 1n, Capacitor_SMD:C_0805_2012Metric_Pad1.18x1.45mm_HandSolder, F.Cu at (273.9, 109.3)
- added C25: 10n, Capacitor_SMD:C_0805_2012Metric_Pad1.18x1.45mm_HandSolder, F.Cu at (259.5, 118.9)
- added C26: 1u, Capacitor_SMD:C_0805_2012Metric_Pad1.18x1.45mm_HandSolder, F.Cu at (269.1, 115.4)
- added C27: 1n, Capacitor_SMD:C_0805_2012Metric_Pad1.18x1.45mm_HandSolder, F.Cu at (269.1, 109.3)
- added C28: 10n, Capacitor_SMD:C_0805_2012Metric_Pad1.18x1.45mm_HandSolder, F.Cu at (269.1, 118.4)
- added C29: 1u, Capacitor_SMD:C_0805_2012Metric_Pad1.18x1.45mm_HandSolder, F.Cu at (269.1, 112.4)
- added C3: 0.1u, Capacitor_SMD:C_0805_2012Metric_Pad1.18x1.45mm_HandSolder, F.Cu at (224.6, 109.3)
- added C30: 1n, Capacitor_SMD:C_0805_2012Metric_Pad1.18x1.45mm_HandSolder, F.Cu at (279.6, 103.3)
- added C31: 0.1u, Capacitor_SMD:C_0805_2012Metric_Pad1.18x1.45mm_HandSolder, F.Cu at (273.9, 115.4)
- added C32: 10n, Capacitor_SMD:C_0805_2012Metric_Pad1.18x1.45mm_HandSolder, F.Cu at (270.0, 103.3)
- added C33: 1u, Capacitor_SMD:C_0805_2012Metric_Pad1.18x1.45mm_HandSolder, F.Cu at (264.3, 109.9)
- added C34: 1u, Capacitor_SMD:C_0805_2012Metric_Pad1.18x1.45mm_HandSolder, F.Cu at (264.3, 106.9)
- added C35: 1u, Capacitor_SMD:C_0805_2012Metric_Pad1.18x1.45mm_HandSolder, F.Cu at (284.4, 103.3)
- added C36: 0.1u, Capacitor_SMD:C_0805_2012Metric_Pad1.18x1.45mm_HandSolder, F.Cu at (269.1, 106.3)
- added C37: 4.7n, Capacitor_SMD:C_0805_2012Metric_Pad1.18x1.45mm_HandSolder, F.Cu at (259.5, 109.9)
- added C38: 0.1u, Capacitor_SMD:C_0805_2012Metric_Pad1.18x1.45mm_HandSolder, F.Cu at (274.8, 103.3)
- added C39: 1u, Capacitor_SMD:C_0805_2012Metric_Pad1.18x1.45mm_HandSolder, F.Cu at (315.3, 84.9)
- added C4: 0.1u, Capacitor_SMD:C_0805_2012Metric_Pad1.18x1.45mm_HandSolder, F.Cu at (229.4, 103.3)
- added C40: 1u, Capacitor_SMD:C_0805_2012Metric_Pad1.18x1.45mm_HandSolder, F.Cu at (325.0, 75.3)
- added C41: 1u, Capacitor_SMD:C_0805_2012Metric_Pad1.18x1.45mm_HandSolder, F.Cu at (315.3, 87.9)
- added C42: 0.1u, Capacitor_SMD:C_0805_2012Metric_Pad1.18x1.45mm_HandSolder, F.Cu at (310.5, 90.9)
- added C43: 0.1u, Capacitor_SMD:C_0805_2012Metric_Pad1.18x1.45mm_HandSolder, F.Cu at (329.8, 75.3)
- added C44: 0.1u, Capacitor_SMD:C_0805_2012Metric_Pad1.18x1.45mm_HandSolder, F.Cu at (310.5, 84.9)
- added C45: 1u, Capacitor_SMD:C_0805_2012Metric_Pad1.18x1.45mm_HandSolder, F.Cu at (310.5, 75.9)
- added C46: 10n, Capacitor_SMD:C_0805_2012Metric_Pad1.18x1.45mm_HandSolder, F.Cu at (315.3, 81.9)
- added C47: 1u, Capacitor_SMD:C_0805_2012Metric_Pad1.18x1.45mm_HandSolder, F.Cu at (334.6, 75.3)
- added C48: 10n, Capacitor_SMD:C_0805_2012Metric_Pad1.18x1.45mm_HandSolder, F.Cu at (325.0, 81.4)
- added C49: 0.1u, Capacitor_SMD:C_0805_2012Metric_Pad1.18x1.45mm_HandSolder, F.Cu at (315.3, 90.9)
- added C5: 0.1u, Capacitor_SMD:C_0805_2012Metric_Pad1.18x1.45mm_HandSolder, F.Cu at (224.6, 103.3)
- added C50: 10n, Capacitor_SMD:C_0805_2012Metric_Pad1.18x1.45mm_HandSolder, F.Cu at (310.5, 81.9)
- added C51: 10n, Capacitor_SMD:C_0805_2012Metric_Pad1.18x1.45mm_HandSolder, F.Cu at (316.2, 72.3)
- added C52: 1u, Capacitor_SMD:C_0805_2012Metric_Pad1.18x1.45mm_HandSolder, F.Cu at (329.8, 78.4)
- added C53: 1n, Capacitor_SMD:C_0805_2012Metric_Pad1.18x1.45mm_HandSolder, F.Cu at (325.0, 78.4)
- added C54: 10n, Capacitor_SMD:C_0805_2012Metric_Pad1.18x1.45mm_HandSolder, F.Cu at (310.5, 87.9)
- added C55: 1u, Capacitor_SMD:C_0805_2012Metric_Pad1.18x1.45mm_HandSolder, F.Cu at (320.2, 84.4)
- added C56: 1n, Capacitor_SMD:C_0805_2012Metric_Pad1.18x1.45mm_HandSolder, F.Cu at (320.2, 78.4)
- added C57: 10n, Capacitor_SMD:C_0805_2012Metric_Pad1.18x1.45mm_HandSolder, F.Cu at (320.2, 87.4)
- added C58: 1u, Capacitor_SMD:C_0805_2012Metric_Pad1.18x1.45mm_HandSolder, F.Cu at (320.2, 81.4)
- added C59: 1n, Capacitor_SMD:C_0805_2012Metric_Pad1.18x1.45mm_HandSolder, F.Cu at (330.6, 72.3)
- added C6: 0.1u, Capacitor_SMD:C_0805_2012Metric_Pad1.18x1.45mm_HandSolder, F.Cu at (229.4, 106.3)
- added C60: 0.1u, Capacitor_SMD:C_0805_2012Metric_Pad1.18x1.45mm_HandSolder, F.Cu at (325.0, 84.4)
- added C61: 10n, Capacitor_SMD:C_0805_2012Metric_Pad1.18x1.45mm_HandSolder, F.Cu at (321.0, 72.3)
- added C62: 1u, Capacitor_SMD:C_0805_2012Metric_Pad1.18x1.45mm_HandSolder, F.Cu at (315.3, 78.9)
- added C63: 1u, Capacitor_SMD:C_0805_2012Metric_Pad1.18x1.45mm_HandSolder, F.Cu at (315.3, 75.9)
- added C64: 1u, Capacitor_SMD:C_0805_2012Metric_Pad1.18x1.45mm_HandSolder, F.Cu at (335.4, 72.3)
- added C65: 0.1u, Capacitor_SMD:C_0805_2012Metric_Pad1.18x1.45mm_HandSolder, F.Cu at (320.2, 75.3)
- added C66: 4.7n, Capacitor_SMD:C_0805_2012Metric_Pad1.18x1.45mm_HandSolder, F.Cu at (310.5, 78.9)
- added C67: 0.1u, Capacitor_SMD:C_0805_2012Metric_Pad1.18x1.45mm_HandSolder, F.Cu at (325.8, 72.3)
- added C68: 10n, Capacitor_SMD:C_0805_2012Metric_Pad1.18x1.45mm_HandSolder, F.Cu at (129.4, 65.8)
- added C69: 0.1u tantalum, Capacitor_SMD:C_0805_2012Metric_Pad1.18x1.45mm_HandSolder, F.Cu at (129.4, 68.8)
- added C7: 10u, Capacitor_SMD:C_0805_2012Metric_Pad1.18x1.45mm_HandSolder, F.Cu at (234.2, 106.3)
- added C70: 0.1u, Capacitor_SMD:C_0805_2012Metric_Pad1.18x1.45mm_HandSolder, F.Cu at (284.5, 137.9)
- added C71: 0.1u, Capacitor_SMD:C_0805_2012Metric_Pad1.18x1.45mm_HandSolder, F.Cu at (284.5, 147.7)
- added C8: 10u, Capacitor_SMD:C_0805_2012Metric_Pad1.18x1.45mm_HandSolder, F.Cu at (224.6, 106.3)
- added C9: 0.1u, Capacitor_SMD:C_0805_2012Metric_Pad1.18x1.45mm_HandSolder, F.Cu at (224.6, 112.4)
- added J1: Conn_02x07_Odd_Even, Connector_IDC:IDC-Header_2x07_P2.54mm_Vertical, F.Cu at (121.8, 116.9)
- added J2: Conn_01x15, centrifuge footprints:L77HDE15SD1CH4FVGA, F.Cu at (242.9, 44.4)
- added J3: Conn_01x15, centrifuge footprints:L77HDE15SD1CH4FVGA, F.Cu at (294.0, 44.4)
- added J4: Conn_01x15, centrifuge footprints:L77HDE15SD1CH4FVGA, F.Cu at (242.9, 75.4)
- added JP1: Jumper_2_Bridged, Jumper:SolderJumper-2_P1.3mm_Bridged_Pad1.0x1.5mm, F.Cu at (257.3, 47.5)
- added JP10: Jumper_2_Bridged, Jumper:SolderJumper-2_P1.3mm_Bridged_Pad1.0x1.5mm, F.Cu at (308.3, 47.5)
- added JP11: SolderJumper_3_Bridged12, Jumper:SolderJumper-3_P1.3mm_Open_Pad1.0x1.5mm_NumberLabels, F.Cu at (134.3, 175.9)
- added JP12: SolderJumper_3_Bridged12, Jumper:SolderJumper-3_P1.3mm_Open_Pad1.0x1.5mm_NumberLabels, F.Cu at (125.9, 185.9)
- added JP13: SolderJumper_3_Bridged12, Jumper:SolderJumper-3_P1.3mm_Open_Pad1.0x1.5mm_NumberLabels, F.Cu at (125.9, 182.4)
- added JP14: SolderJumper_3_Bridged12, Jumper:SolderJumper-3_P1.3mm_Open_Pad1.0x1.5mm_NumberLabels, F.Cu at (345.9, 67.9)
- added JP15: Jumper_2_Bridged, Jumper:SolderJumper-2_P1.3mm_Bridged_Pad1.0x1.5mm, F.Cu at (350.9, 67.9)
- added JP16: Jumper_2_Bridged, Jumper:SolderJumper-2_P1.3mm_Bridged_Pad1.0x1.5mm, F.Cu at (345.3, 71.5)
- added JP17: Jumper_2_Bridged, Jumper:SolderJumper-2_P1.3mm_Bridged_Pad1.0x1.5mm, F.Cu at (257.3, 78.5)
- added JP18: SolderJumper_3_Bridged12, Jumper:SolderJumper-3_P1.3mm_Open_Pad1.0x1.5mm_NumberLabels, F.Cu at (114.0, 155.6)
- added JP19: SolderJumper_3_Bridged12, Jumper:SolderJumper-3_P1.3mm_Open_Pad1.0x1.5mm_NumberLabels, F.Cu at (111.2, 162.0)
- added JP20: SolderJumper_3_Bridged12, Jumper:SolderJumper-3_P1.3mm_Open_Pad1.0x1.5mm_NumberLabels, F.Cu at (105.5, 162.0)
- added JP21: SolderJumper_3_Bridged12, Jumper:SolderJumper-3_P1.3mm_Open_Pad1.0x1.5mm_NumberLabels, F.Cu at (276.0, 72.6)
- added JP22: Jumper_2_Bridged, Jumper:SolderJumper-2_P1.3mm_Bridged_Pad1.0x1.5mm, F.Cu at (281.0, 72.6)
- added JP23: Jumper_2_Bridged, Jumper:SolderJumper-2_P1.3mm_Bridged_Pad1.0x1.5mm, F.Cu at (275.4, 76.2)
- added JP8: Jumper_3_Open, Jumper:SolderJumper-3_P1.3mm_Open_Pad1.0x1.5mm_NumberLabels, F.Cu at (259.9, 103.6)
- added JP9: Jumper_3_Open, Jumper:SolderJumper-3_P1.3mm_Open_Pad1.0x1.5mm_NumberLabels, F.Cu at (311.0, 72.6)
- added Q1: BSN20, Package_TO_SOT_SMD:SOT-23, F.Cu at (162.7, 129.9)
- added Q2: BSN20, Package_TO_SOT_SMD:SOT-23, F.Cu at (157.2, 133.5)
- added Q3: BSN20, Package_TO_SOT_SMD:SOT-23, F.Cu at (134.2, 156.0)
- added Q4: BSN20, Package_TO_SOT_SMD:SOT-23, F.Cu at (128.7, 159.6)
- added Q5: BSN20, Package_TO_SOT_SMD:SOT-23, F.Cu at (110.7, 170.6)
- added Q6: BSN20, Package_TO_SOT_SMD:SOT-23, F.Cu at (105.1, 174.1)
- added R1: 4.7k, Resistor_SMD:R_0805_2012Metric_Pad1.20x1.40mm_HandSolder, F.Cu at (326.6, 44.3)
- added R10: 330, Resistor_SMD:R_0805_2012Metric_Pad1.20x1.40mm_HandSolder, F.Cu at (294.4, 104.5)
- added R11: 4.7k, Resistor_SMD:R_0805_2012Metric_Pad1.20x1.40mm_HandSolder, F.Cu at (294.4, 98.6)
- added R12: vga_ddc_sda_pullup_l, Resistor_SMD:R_0805_2012Metric_Pad1.20x1.40mm_HandSolder, F.Cu at (257.5, 44.3)
- added R13: vga_ddc_scl_pullup_l, Resistor_SMD:R_0805_2012Metric_Pad1.20x1.40mm_HandSolder, F.Cu at (224.5, 65.6)
- added R14: vga_ddc_sda_pullup_h, Resistor_SMD:R_0805_2012Metric_Pad1.20x1.40mm_HandSolder, F.Cu at (234.0, 65.6)
- added R15: vga_ddc_scl_pullup_h, Resistor_SMD:R_0805_2012Metric_Pad1.20x1.40mm_HandSolder, F.Cu at (229.3, 65.6)
- added R16: 1k, Resistor_SMD:R_0805_2012Metric_Pad1.20x1.40mm_HandSolder, F.Cu at (262.2, 41.3)
- added R17: 1k, Resistor_SMD:R_0805_2012Metric_Pad1.20x1.40mm_HandSolder, F.Cu at (257.5, 41.3)
- added R18: 1k, Resistor_SMD:R_0805_2012Metric_Pad1.20x1.40mm_HandSolder, F.Cu at (361.5, 41.3)
- added R19: 1k, Resistor_SMD:R_0805_2012Metric_Pad1.20x1.40mm_HandSolder, F.Cu at (361.5, 44.3)
- added R2: 4.7k, Resistor_SMD:R_0805_2012Metric_Pad1.20x1.40mm_HandSolder, F.Cu at (326.6, 41.3)
- added R20: 1k, Resistor_SMD:R_0805_2012Metric_Pad1.20x1.40mm_HandSolder, F.Cu at (366.3, 41.3)
- added R21: 1k, Resistor_SMD:R_0805_2012Metric_Pad1.20x1.40mm_HandSolder, F.Cu at (366.3, 44.3)
- added R22: 1.5k, Resistor_SMD:R_0805_2012Metric_Pad1.20x1.40mm_HandSolder, F.Cu at (278.7, 112.3)
- added R23: 2.2k, Resistor_SMD:R_0805_2012Metric_Pad1.20x1.40mm_HandSolder, F.Cu at (283.5, 109.3)
- added R24: 2.2k, Resistor_SMD:R_0805_2012Metric_Pad1.20x1.40mm_HandSolder, F.Cu at (269.1, 121.4)
- added R25: 2.2k, Resistor_SMD:R_0805_2012Metric_Pad1.20x1.40mm_HandSolder, F.Cu at (273.9, 118.3)
- added R26: 2.2k, Resistor_SMD:R_0805_2012Metric_Pad1.20x1.40mm_HandSolder, F.Cu at (278.7, 115.3)
- added R27: 1.5k, Resistor_SMD:R_0805_2012Metric_Pad1.20x1.40mm_HandSolder, F.Cu at (329.7, 81.3)
- added R28: 2.2k, Resistor_SMD:R_0805_2012Metric_Pad1.20x1.40mm_HandSolder, F.Cu at (334.6, 78.3)
- added R29: 2.2k, Resistor_SMD:R_0805_2012Metric_Pad1.20x1.40mm_HandSolder, F.Cu at (320.1, 90.4)
- added R3: 75, Resistor_SMD:R_0805_2012Metric_Pad1.20x1.40mm_HandSolder, F.Cu at (224.5, 118.3)
- added R30: 2.2k, Resistor_SMD:R_0805_2012Metric_Pad1.20x1.40mm_HandSolder, F.Cu at (324.9, 87.4)
- added R31: 2.2k, Resistor_SMD:R_0805_2012Metric_Pad1.20x1.40mm_HandSolder, F.Cu at (329.7, 84.3)
- added R32: vga_ddc_sda_pullup_l, Resistor_SMD:R_0805_2012Metric_Pad1.20x1.40mm_HandSolder, F.Cu at (308.5, 44.3)
- added R33: vga_ddc_scl_pullup_l, Resistor_SMD:R_0805_2012Metric_Pad1.20x1.40mm_HandSolder, F.Cu at (275.6, 65.6)
- added R34: vga_ddc_sda_pullup_h, Resistor_SMD:R_0805_2012Metric_Pad1.20x1.40mm_HandSolder, F.Cu at (285.1, 65.6)
- added R35: vga_ddc_scl_pullup_h, Resistor_SMD:R_0805_2012Metric_Pad1.20x1.40mm_HandSolder, F.Cu at (280.3, 65.6)
- added R36: 1k, Resistor_SMD:R_0805_2012Metric_Pad1.20x1.40mm_HandSolder, F.Cu at (313.3, 41.3)
- added R37: 1k, Resistor_SMD:R_0805_2012Metric_Pad1.20x1.40mm_HandSolder, F.Cu at (308.5, 41.3)
- added R38: vga_ddc_sda_pullup_l, Resistor_SMD:R_0805_2012Metric_Pad1.20x1.40mm_HandSolder, F.Cu at (257.5, 75.3)
- added R39: vga_ddc_scl_pullup_l, Resistor_SMD:R_0805_2012Metric_Pad1.20x1.40mm_HandSolder, F.Cu at (224.5, 96.6)
- added R4: 75, Resistor_SMD:R_0805_2012Metric_Pad1.20x1.40mm_HandSolder, F.Cu at (234.2, 109.3)
- added R40: vga_ddc_sda_pullup_h, Resistor_SMD:R_0805_2012Metric_Pad1.20x1.40mm_HandSolder, F.Cu at (234.0, 96.6)
- added R41: vga_ddc_scl_pullup_h, Resistor_SMD:R_0805_2012Metric_Pad1.20x1.40mm_HandSolder, F.Cu at (229.3, 96.6)
- added R42: 1k, Resistor_SMD:R_0805_2012Metric_Pad1.20x1.40mm_HandSolder, F.Cu at (262.2, 72.3)
- added R43: 1k, Resistor_SMD:R_0805_2012Metric_Pad1.20x1.40mm_HandSolder, F.Cu at (257.5, 72.3)
- added R44: 10k, Resistor_SMD:R_0805_2012Metric_Pad1.20x1.40mm_HandSolder, F.Cu at (129.4, 62.8)
- added R45: 10k, Resistor_SMD:R_0805_2012Metric_Pad1.20x1.40mm_HandSolder, F.Cu at (284.5, 140.9)
- added R46: 10k, Resistor_SMD:R_0805_2012Metric_Pad1.20x1.40mm_HandSolder, F.Cu at (284.5, 150.7)
- added R5: 75, Resistor_SMD:R_0805_2012Metric_Pad1.20x1.40mm_HandSolder, F.Cu at (239.0, 103.3)
- added R6: 3.8k, Resistor_SMD:R_0805_2012Metric_Pad1.20x1.40mm_HandSolder, F.Cu at (229.3, 112.3)
- added R7: 2.2k, Resistor_SMD:R_0805_2012Metric_Pad1.20x1.40mm_HandSolder, F.Cu at (224.5, 115.3)
- added R8: 10k, Resistor_SMD:R_0805_2012Metric_Pad1.20x1.40mm_HandSolder, F.Cu at (299.2, 98.6)
- added R9: 10k, Resistor_SMD:R_0805_2012Metric_Pad1.20x1.40mm_HandSolder, F.Cu at (294.4, 101.6)
- added U10: M24C02-WMN, Package_SO:SOIC-8_3.9x4.9mm_P1.27mm, F.Cu at (127.3, 177.4)
- added U11: LSF0102, Package_SO:VSSOP-8_2.3x2mm_P0.5mm, F.Cu at (105.5, 170.1)
- added U12: M24C02-WMN, Package_SO:SOIC-8_3.9x4.9mm_P1.27mm, F.Cu at (106.9, 157.0)
- added U4: TVP7002, Package_QFP:TQFP-100-1EP_14x14mm_P0.5mm_EP5x5mm_ThermalVias, F.Cu at (89.3, 57.0)
- added U5: THS8136, Package_QFP:LQFP-48-1EP_7x7mm_P0.5mm_EP3.6x3.6mm, F.Cu at (183.9, 118.8)
- added U6: LSF0102, Package_SO:VSSOP-8_2.3x2mm_P0.5mm, F.Cu at (157.5, 129.5)
- added U8: TVP7002, Package_QFP:TQFP-100-1EP_14x14mm_P0.5mm_EP5x5mm_ThermalVias, F.Cu at (74.5, 119.3)
- added U9: LSF0102, Package_SO:VSSOP-8_2.3x2mm_P0.5mm, F.Cu at (129.0, 155.6)
- added X1: ECS-2333-270-BN, Oscillator:Oscillator_SMD_EuroQuartz_XO32-4Pin_3.2x2.5mm_HandSoldering, F.Cu at (90.7, 155.8)
- added X2: ECS-2333-270-BN, Oscillator:Oscillator_SMD_EuroQuartz_XO32-4Pin_3.2x2.5mm_HandSoldering, F.Cu at (90.7, 179.7)
- added X3: EC2620TTS-100.000MTR, Oscillator:Oscillator_SMD_EuroQuartz_XO91-4Pin_7.0x5.0mm_HandSoldering, F.Cu at (137.6, 66.4)
Connections:
- net /fpga_core/config_dram/CCLK renamed /config_sram/CCLK
- net /fpga_core/config_dram/SRAM_A10 renamed /config_sram/SRAM_A10
- net /fpga_core/config_dram/SRAM_A11 renamed /config_sram/SRAM_A11
- net /fpga_core/config_dram/SRAM_A12 renamed /config_sram/SRAM_A12
- net /fpga_core/config_dram/SRAM_A13 renamed /config_sram/SRAM_A13
- net /fpga_core/config_dram/SRAM_A14 renamed /config_sram/SRAM_A14
- net /fpga_core/config_dram/SRAM_A2 renamed /config_sram/SRAM_A2
- net /fpga_core/config_dram/SRAM_A3 renamed /config_sram/SRAM_A3
- net /fpga_core/config_dram/SRAM_A4 renamed /config_sram/SRAM_A4
- net /fpga_core/config_dram/SRAM_A5 renamed /config_sram/SRAM_A5
- net /fpga_core/config_dram/SRAM_A6 renamed /config_sram/SRAM_A6
- net /fpga_core/config_dram/SRAM_A9 renamed /config_sram/SRAM_A9
- net /fpga_core/config_dram/SRAM_ADV_LD renamed /config_sram/SRAM_ADV_LD
- net /fpga_core/config_dram/SRAM_CE1 renamed /config_sram/SRAM_CE1
- net /fpga_core/config_dram/SRAM_CE2 renamed /config_sram/SRAM_CE2
- net /fpga_core/config_dram/SRAM_CLK renamed /config_sram/SRAM_CLK
- net /fpga_core/config_dram/SRAM_D0 renamed /config_sram/SRAM_D0
- net /fpga_core/config_dram/SRAM_D1 renamed /config_sram/SRAM_D1
- net /fpga_core/config_dram/SRAM_D10 renamed /config_sram/SRAM_D10
- net /fpga_core/config_dram/SRAM_D11 renamed /config_sram/SRAM_D11
- net /fpga_core/config_dram/SRAM_D12 renamed /config_sram/SRAM_D12
- net /fpga_core/config_dram/SRAM_D13 renamed /config_sram/SRAM_D13
- net /fpga_core/config_dram/SRAM_D14 renamed /config_sram/SRAM_D14
- net /fpga_core/config_dram/SRAM_D15 renamed /config_sram/SRAM_D15
- net /fpga_core/config_dram/SRAM_D16 renamed /config_sram/SRAM_D16
- net /fpga_core/config_dram/SRAM_D18 renamed /config_sram/SRAM_D18
- net /fpga_core/config_dram/SRAM_D20 renamed /config_sram/SRAM_D20
- net /fpga_core/config_dram/SRAM_D21 renamed /config_sram/SRAM_D21
- net /fpga_core/config_dram/SRAM_D22 renamed /config_sram/SRAM_D22
- net /fpga_core/config_dram/SRAM_D23 renamed /config_sram/SRAM_D23
- net /fpga_core/config_dram/SRAM_D24 renamed /config_sram/SRAM_D24
- net /fpga_core/config_dram/SRAM_D25 renamed /config_sram/SRAM_D25
- net /fpga_core/config_dram/SRAM_D26 renamed /config_sram/SRAM_D26
- net /fpga_core/config_dram/SRAM_D27 renamed /config_sram/SRAM_D27
- net /fpga_core/config_dram/SRAM_D28 renamed /config_sram/SRAM_D28
- net /fpga_core/config_dram/SRAM_D29 renamed /config_sram/SRAM_D29
- net /fpga_core/config_dram/SRAM_D30 renamed /config_sram/SRAM_D30
- net /fpga_core/config_dram/SRAM_D31 renamed /config_sram/SRAM_D31
- net /fpga_core/config_dram/SRAM_D32 renamed /config_sram/SRAM_D32
- net /fpga_core/config_dram/SRAM_D33 renamed /config_sram/SRAM_D33
- net /fpga_core/config_dram/SRAM_D34 renamed /config_sram/SRAM_D34
- net /fpga_core/config_dram/SRAM_D35 renamed /config_sram/SRAM_D35
- net /fpga_core/config_dram/SRAM_D4 renamed /config_sram/SRAM_D4
- net /fpga_core/config_dram/SRAM_D5 renamed /config_sram/SRAM_D5
- net /fpga_core/config_dram/SRAM_D6 renamed /config_sram/SRAM_D6
- net /fpga_core/config_dram/SRAM_D8 renamed /config_sram/SRAM_D8
- net /fpga_core/config_dram/SRAM_D9 renamed /config_sram/SRAM_D9
- net /fpga_core/config_dram/SRAM_OE renamed /config_sram/SRAM_OE
- net /fpga_core/config_dram/SRAM_WE renamed /config_sram/SRAM_WE
- net Net-(R5-Pad2) renamed /config_sram/IO2
- net Net-(R6-Pad2) renamed /config_sram/IO3
- net Net-(U1-PadJ13) renamed /config_sram/IO0
- net Net-(U1-PadJ14) renamed /config_sram/IO1
- net Net-(U1-PadL12) renamed /config_sram/n_CONFIG_CS
- U1 pad A10: /fpga_core/config_dram/SRAM_A0 -> /config_sram/SRAM_A1
- U1 pad A12: /fpga_core/config_dram/SRAM_A0 -> /config_sram/SRAM_A20
- U1 pad A13: /fpga_core/config_dram/SRAM_A7 -> /config_sram/SRAM_A7
- U1 pad A14: /fpga_core/config_dram/SRAM_A8 -> /config_sram/SRAM_A8
- U1 pad A16: unconnected-(U1-PadA16) -> +3.3VA
- U1 pad A3: unconnected-(U1-PadA3) -> /fpga_core/IN0.G6
- U1 pad A4: unconnected-(U1-PadA4) -> /fpga_core/IN0.G8
- U1 pad A5: unconnected-(U1-PadA5) -> /fpga_core/IN0.G9
- U1 pad A6: unconnected-(U1-PadA6) -> +3.3VA
- U1 pad A7: unconnected-(U1-PadA7) -> /fpga_core/IN0.R7
- U1 pad A8: /fpga_core/config_dram/SRAM_A16 -> unconnected-(U1-PadA8)
- U1 pad A9: /fpga_core/config_dram/SRAM_A15 -> unconnected-(U1-PadA9)
- U1 pad B1: unconnected-(U1-PadB1) -> /fpga_core/FIDIN0
- U1 pad B10: unconnected-(U1-PadB10) -> /config_sram/SRAM_A0
- U1 pad B11: /fpga_core/config_dram/SRAM_A1 -> /config_sram/SRAM_A19
- U1 pad B13: unconnected-(U1-PadB13) -> +3.3VA
- U1 pad B2: unconnected-(U1-PadB2) -> /fpga_core/IN0.B5
- U1 pad B3: unconnected-(U1-PadB3) -> +3.3VA
- U1 pad B4: unconnected-(U1-PadB4) -> /fpga_core/IN0.G7
- U1 pad B5: unconnected-(U1-PadB5) -> /fpga_core/IN0.R5
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Routing:
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- added copper zone on In6.Cu, net +3.3VA
- added copper zone on In1.Cu, net GND

Commit message: FPGA PCB design completed
Parts:
- added C100: 470n, Capacitor_SMD:C_0603_1608Metric_Pad1.08x0.95mm_HandSolder, B.Cu at (139.2, 71.4)
- added C101: 470n, Capacitor_SMD:C_0603_1608Metric_Pad1.08x0.95mm_HandSolder, B.Cu at (138.6, 98.5)
- added C102: 470n, Capacitor_SMD:C_0603_1608Metric_Pad1.08x0.95mm_HandSolder, B.Cu at (142.9, 71.5)
- added C103: 470n, Capacitor_SMD:C_0603_1608Metric_Pad1.08x0.95mm_HandSolder, B.Cu at (139.0, 81.3)
- added C104: 4.7u, Capacitor_SMD:C_0805_2012Metric_Pad1.18x1.45mm_HandSolder, B.Cu at (114.5, 86.3)
- added C105: 4.7u, Capacitor_SMD:C_0805_2012Metric_Pad1.18x1.45mm_HandSolder, B.Cu at (120.8, 74.6)
- added C106: 4.7u, Capacitor_SMD:C_0805_2012Metric_Pad1.18x1.45mm_HandSolder, B.Cu at (140.0, 76.7)
- added C107: 4.7u, Capacitor_SMD:C_0805_2012Metric_Pad1.18x1.45mm_HandSolder, B.Cu at (121.8, 78.1)
- added C108: 47u X5R/X7R, Capacitor_SMD:C_1210_3225Metric_Pad1.33x2.70mm_HandSolder, B.Cu at (119.5, 100.3)
- added C109: 470n, Capacitor_SMD:C_0603_1608Metric_Pad1.08x0.95mm_HandSolder, B.Cu at (119.3, 104.7)
- added C110: 470n, Capacitor_SMD:C_0603_1608Metric_Pad1.08x0.95mm_HandSolder, B.Cu at (138.5, 83.1)
- added C111: 470n, Capacitor_SMD:C_0603_1608Metric_Pad1.08x0.95mm_HandSolder, B.Cu at (140.8, 78.5)
- added C112: 470n, Capacitor_SMD:C_0603_1608Metric_Pad1.08x0.95mm_HandSolder, B.Cu at (140.6, 100.7)
- added C113: 470n, Capacitor_SMD:C_0603_1608Metric_Pad1.08x0.95mm_HandSolder, F.Cu at (119.2, 102.8)
- added C114: 470n, Capacitor_SMD:C_0603_1608Metric_Pad1.08x0.95mm_HandSolder, B.Cu at (124.7, 78.8)
- added C115: 470n, Capacitor_SMD:C_0603_1608Metric_Pad1.08x0.95mm_HandSolder, B.Cu at (125.6, 100.6)
- added C116: 470n, Capacitor_SMD:C_0603_1608Metric_Pad1.08x0.95mm_HandSolder, B.Cu at (139.2, 92.9)
- added C117: 4.7u, Capacitor_SMD:C_0805_2012Metric_Pad1.18x1.45mm_HandSolder, B.Cu at (125.4, 75.2)
- added C118: 4.7u, Capacitor_SMD:C_0805_2012Metric_Pad1.18x1.45mm_HandSolder, B.Cu at (129.0, 97.8)
- added C119: 4.7u, Capacitor_SMD:C_0805_2012Metric_Pad1.18x1.45mm_HandSolder, B.Cu at (140.1, 88.7)
- added C120: 4.7u, Capacitor_SMD:C_0805_2012Metric_Pad1.18x1.45mm_HandSolder, B.Cu at (116.3, 82.6)
- added C121: 47u X5R/X7R, Capacitor_SMD:C_1210_3225Metric_Pad1.33x2.70mm_HandSolder, B.Cu at (128.7, 105.0)
- added C122: 47u X5R/X7R, Capacitor_SMD:C_1210_3225Metric_Pad1.33x2.70mm_HandSolder, B.Cu at (113.5, 81.6)
- added C123: 0.1u, Capacitor_SMD:C_0805_2012Metric_Pad1.18x1.45mm_HandSolder, B.Cu at (145.9, 81.2)
- added C124: 0.1u, Capacitor_SMD:C_0805_2012Metric_Pad1.18x1.45mm_HandSolder, B.Cu at (149.9, 81.2)
- added C125: 0.1u, Capacitor_SMD:C_0805_2012Metric_Pad1.18x1.45mm_HandSolder, B.Cu at (147.4, 83.4)
- added C126: 0.1u, Capacitor_SMD:C_0805_2012Metric_Pad1.18x1.45mm_HandSolder, B.Cu at (148.1, 89.8)
- added C127: 0.1u, Capacitor_SMD:C_0805_2012Metric_Pad1.18x1.45mm_HandSolder, B.Cu at (152.3, 93.1)
- added C128: 0.1u, Capacitor_SMD:C_0805_2012Metric_Pad1.18x1.45mm_HandSolder, B.Cu at (147.9, 93.2)
- added C129: 0.1u, Capacitor_SMD:C_0805_2012Metric_Pad1.18x1.45mm_HandSolder, B.Cu at (152.2, 85.7)
- added C130: 0.1u, Capacitor_SMD:C_0805_2012Metric_Pad1.18x1.45mm_HandSolder, B.Cu at (147.8, 96.0)
- added C131: 0.1u, Capacitor_SMD:C_0805_2012Metric_Pad1.18x1.45mm_HandSolder, B.Cu at (152.3, 89.7)
- added C132: 0.1u, Capacitor_SMD:C_0805_2012Metric_Pad1.18x1.45mm_HandSolder, B.Cu at (147.6, 85.8)
- added C133: 0.1u, Capacitor_SMD:C_0805_2012Metric_Pad1.18x1.45mm_HandSolder, B.Cu at (152.3, 95.9)
- added C134: 0.1u, Capacitor_SMD:C_0805_2012Metric_Pad1.18x1.45mm_HandSolder, B.Cu at (151.7, 83.5)
- added C72: 47u X5R/X7R, Capacitor_SMD:C_1210_3225Metric_Pad1.33x2.70mm_HandSolder, B.Cu at (113.9, 97.6)
- added C73: 4.7u, Capacitor_SMD:C_0805_2012Metric_Pad1.18x1.45mm_HandSolder, B.Cu at (134.4, 97.9)
- added C74: 100u tantalum 1-40 mOhm or X5R/X7R, Capacitor_SMD:C_1210_3225Metric_Pad1.33x2.70mm_HandSolder, B.Cu at (136.2, 85.6)
- added C75: 4.7u, Capacitor_SMD:C_0805_2012Metric_Pad1.18x1.45mm_HandSolder, B.Cu at (118.4, 97.1)
- added C76: 470n, Capacitor_SMD:C_0603_1608Metric_Pad1.08x0.95mm_HandSolder, B.Cu at (117.7, 94.9)
- added C77: 470n, Capacitor_SMD:C_0603_1608Metric_Pad1.08x0.95mm_HandSolder, B.Cu at (128.4, 87.0)
- added C78: 470n, Capacitor_SMD:C_0603_1608Metric_Pad1.08x0.95mm_HandSolder, B.Cu at (135.9, 88.0)
- added C79: 470n, Capacitor_SMD:C_0603_1608Metric_Pad1.08x0.95mm_HandSolder, B.Cu at (127.5, 78.2)
- added C80: 470n, Capacitor_SMD:C_0603_1608Metric_Pad1.08x0.95mm_HandSolder, B.Cu at (134.9, 89.5)
- added C81: 470n, Capacitor_SMD:C_0603_1608Metric_Pad1.08x0.95mm_HandSolder, B.Cu at (128.1, 76.6)
- added C82: 330u tantalum 5-40 mOhm, Capacitor_Tantalum_SMD:CP_EIA-7343-31_Kemet-D_Pad2.25x2.55mm_HandSolder, B.Cu at (130.7, 81.5)
- added C83: 470n, Capacitor_SMD:C_0603_1608Metric_Pad1.08x0.95mm_HandSolder, B.Cu at (124.2, 87.0)
- added C84: 4.7u, Capacitor_SMD:C_0805_2012Metric_Pad1.18x1.45mm_HandSolder, B.Cu at (134.4, 99.9)
- added C85: 470n, Capacitor_SMD:C_0603_1608Metric_Pad1.08x0.95mm_HandSolder, B.Cu at (135.6, 93.9)
- added C86: 4.7u, Capacitor_SMD:C_0805_2012Metric_Pad1.18x1.45mm_HandSolder, B.Cu at (126.9, 89.2)
- added C87: 470n, Capacitor_SMD:C_0603_1608Metric_Pad1.08x0.95mm_HandSolder, B.Cu at (119.5, 90.4)
- added C88: 4.7u, Capacitor_SMD:C_0805_2012Metric_Pad1.18x1.45mm_HandSolder, B.Cu at (115.1, 101.2)
- added C89: 470n, Capacitor_SMD:C_0603_1608Metric_Pad1.08x0.95mm_HandSolder, B.Cu at (119.6, 85.9)
- added C90: 4.7u, Capacitor_SMD:C_0805_2012Metric_Pad1.18x1.45mm_HandSolder, B.Cu at (118.4, 93.1)
- added C91: 470n, Capacitor_SMD:C_0603_1608Metric_Pad1.08x0.95mm_HandSolder, B.Cu at (135.2, 92.4)
- added C92: 4.7u, Capacitor_SMD:C_0805_2012Metric_Pad1.18x1.45mm_HandSolder, B.Cu at (118.8, 87.6)
- added C93: 470n, Capacitor_SMD:C_0603_1608Metric_Pad1.08x0.95mm_HandSolder, B.Cu at (130.8, 100.0)
- added C94: 4.7u, Capacitor_SMD:C_0805_2012Metric_Pad1.18x1.45mm_HandSolder, B.Cu at (123.7, 97.2)
- added C95: 470n, Capacitor_SMD:C_0603_1608Metric_Pad1.08x0.95mm_HandSolder, B.Cu at (134.6, 95.5)
- added C96: 470n, Capacitor_SMD:C_0603_1608Metric_Pad1.08x0.95mm_HandSolder, B.Cu at (114.7, 90.0)
- added C97: 470n, Capacitor_SMD:C_0603_1608Metric_Pad1.08x0.95mm_HandSolder, B.Cu at (121.7, 76.4)
- added C98: 470n, Capacitor_SMD:C_0603_1608Metric_Pad1.08x0.95mm_HandSolder, B.Cu at (118.0, 77.3)
- added C99: 470n, Capacitor_SMD:C_0603_1608Metric_Pad1.08x0.95mm_HandSolder, B.Cu at (146.4, 71.4)
- added J5: Conn_02x12_Odd_Even, Connector_PinHeader_2.54mm:PinHeader_2x12_P2.54mm_Horizontal, F.Cu at (188.3, 78.2)
- added J6: Conn_02x12_Odd_Even, Connector_PinHeader_2.54mm:PinHeader_2x12_P2.54mm_Horizontal, F.Cu at (213.8, 110.6)
- added R47: 4.7k, Resistor_SMD:R_0805_2012Metric_Pad1.20x1.40mm_HandSolder, F.Cu at (162.1, 102.7)
- added R48: 75, Resistor_SMD:R_0805_2012Metric_Pad1.20x1.40mm_HandSolder, B.Cu at (83.8, 65.5)
- added R49: 75, Resistor_SMD:R_0805_2012Metric_Pad1.20x1.40mm_HandSolder, B.Cu at (83.8, 59.6)
- added R50: 75, Resistor_SMD:R_0805_2012Metric_Pad1.20x1.40mm_HandSolder, B.Cu at (81.7, 68.8)
- added R51: 75, Resistor_SMD:R_0805_2012Metric_Pad1.20x1.40mm_HandSolder, B.Cu at (83.7, 96.9)
- added R52: 75, Resistor_SMD:R_0805_2012Metric_Pad1.20x1.40mm_HandSolder, B.Cu at (83.8, 92.2)
- added R53: 75, Resistor_SMD:R_0805_2012Metric_Pad1.20x1.40mm_HandSolder, B.Cu at (80.4, 101.1)
- added R54: 330, Resistor_SMD:R_0805_2012Metric_Pad1.20x1.40mm_HandSolder, F.Cu at (134.2, 109.1)
- added SW1: SW_MEC_5E, centrifuge footprints:SW_Push_1P1T_NO_6x6mm_H9.5mm_modified, F.Cu at (131.1, 114.8)
- added TP10: TestPoint, TestPoint:TestPoint_Keystone_5015_Micro-Minature, F.Cu at (96.3, 75.1)
- added TP11: TestPoint, TestPoint:TestPoint_Keystone_5015_Micro-Minature, F.Cu at (87.3, 112.8)
- added TP12: TestPoint, TestPoint:TestPoint_Keystone_5015_Micro-Minature, F.Cu at (87.3, 115.6)
- added TP13: TestPoint, TestPoint:TestPoint_Keystone_5015_Micro-Minature, F.Cu at (109.6, 99.8)
- added TP14: TestPoint, TestPoint:TestPoint_Keystone_5015_Micro-Minature, F.Cu at (129.7, 55.1)
- added TP15: TestPoint, TestPoint:TestPoint_Keystone_5015_Micro-Minature, B.Cu at (121.7, 80.5)
- added TP16: TestPoint, TestPoint:TestPoint_Keystone_5015_Micro-Minature, F.Cu at (162.8, 83.7)
- added TP17: TestPoint, TestPoint:TestPoint_Keystone_5015_Micro-Minature, F.Cu at (126.7, 104.0)
- added TP18: TestPoint, TestPoint:TestPoint_Keystone_5015_Micro-Minature, F.Cu at (130.0, 109.9)
- added TP19: TestPoint, TestPoint:TestPoint_Keystone_5015_Micro-Minature, B.Cu at (134.7, 102.4)
- added TP2: TestPoint, TestPoint:TestPoint_Keystone_5015_Micro-Minature, F.Cu at (122.6, 67.3)
- added TP20: TestPoint, TestPoint:TestPoint_Keystone_5015_Micro-Minature, F.Cu at (87.4, 135.6)
- added TP21: TestPoint, TestPoint:TestPoint_Keystone_5015_Micro-Minature, F.Cu at (88.7, 126.8)
- added TP22: TestPoint, TestPoint:TestPoint_Keystone_5015_Micro-Minature, F.Cu at (87.2, 121.2)
- added TP23: TestPoint, TestPoint:TestPoint_Keystone_5015_Micro-Minature, F.Cu at (87.3, 118.4)
- added TP24: TestPoint, TestPoint:TestPoint_Keystone_5015_Micro-Minature, F.Cu at (87.2, 132.6)
- added TP25: TestPoint, TestPoint:TestPoint_Keystone_5015_Micro-Minature, F.Cu at (87.2, 129.6)
- added TP26: TestPoint, TestPoint:TestPoint_Keystone_5015_Micro-Minature, F.Cu at (87.2, 124.0)
- added TP27: TestPoint, TestPoint:TestPoint_Keystone_5015_Micro-Minature, F.Cu at (86.5, 105.1)
- added TP28: TestPoint, TestPoint:TestPoint_Keystone_5015_Micro-Minature, F.Cu at (86.6, 84.4)
- added TP29: TestPoint, TestPoint:TestPoint_Keystone_5015_Micro-Minature, F.Cu at (86.5, 79.8)
- added TP3: TestPoint, TestPoint:TestPoint_Keystone_5015_Micro-Minature, F.Cu at (129.2, 63.2)
- added TP30: TestPoint, TestPoint:TestPoint_Keystone_5015_Micro-Minature, F.Cu at (87.4, 75.8)
- added TP31: TestPoint, TestPoint:TestPoint_Keystone_5015_Micro-Minature, F.Cu at (86.4, 98.3)
- added TP32: TestPoint, TestPoint:TestPoint_Keystone_5015_Micro-Minature, F.Cu at (87.2, 94.8)
- added TP33: TestPoint, TestPoint:TestPoint_Keystone_5015_Micro-Minature, F.Cu at (87.2, 92.0)
- added TP34: TestPoint, TestPoint:TestPoint_Keystone_5015_Micro-Minature, B.Cu at (68.0, 82.5)
- added TP35: TestPoint, TestPoint:TestPoint_Keystone_5015_Micro-Minature, B.Cu at (65.1, 99.2)
- added TP36: TestPoint, TestPoint:TestPoint_Keystone_5015_Micro-Minature, F.Cu at (93.6, 70.5)
- added TP37: TestPoint, TestPoint:TestPoint_Keystone_5015_Micro-Minature, F.Cu at (98.8, 55.7)
- added TP38: TestPoint, TestPoint:TestPoint_Keystone_5015_Micro-Minature, F.Cu at (99.2, 58.5)
- added TP39: TestPoint, TestPoint:TestPoint_Keystone_5015_Micro-Minature, F.Cu at (93.6, 53.0)
- added TP4: TestPoint, TestPoint:TestPoint_Keystone_5015_Micro-Minature, F.Cu at (129.2, 58.8)
- added TP40: TestPoint, TestPoint:TestPoint_Keystone_5015_Micro-Minature, F.Cu at (93.7, 65.6)
- added TP41: TestPoint, TestPoint:TestPoint_Keystone_5015_Micro-Minature, F.Cu at (93.7, 62.9)
- added TP42: TestPoint, TestPoint:TestPoint_Keystone_5015_Micro-Minature, F.Cu at (93.6, 58.0)
- added TP43: TestPoint, TestPoint:TestPoint_Keystone_5015_Micro-Minature, B.Cu at (73.3, 49.4)
- added TP44: TestPoint, TestPoint:TestPoint_Keystone_5015_Micro-Minature, B.Cu at (85.3, 56.3)
- added U13: PESD4USB5B-TTS, Package_DFN_QFN:Diodes_UDFN-10_1.0x2.5mm_P0.5mm, B.Cu at (72.0, 92.0)
- added U14: PESD4USB5B-TTS, Package_DFN_QFN:Diodes_UDFN-10_1.0x2.5mm_P0.5mm, B.Cu at (69.9, 59.9)
- added U15: D5V0FS4U10LP, Package_DFN_QFN:Diodes_UDFN-10_1.0x2.5mm_P0.5mm, F.Cu at (99.3, 130.8)
- added U7: PESD4USB5B-TTS, Package_DFN_QFN:Diodes_UDFN-10_1.0x2.5mm_P0.5mm, B.Cu at (71.3, 123.9)
- C1, C10, C11, C12, C16, C18, C2, C20, C23, C24, C26, C27, C29, C30, C31, C33, C34, C35, C36, C39, C40, C41, C45, C46, C47, C49, C53, C55, C56, C58, C59, C60, C62, C63, C64, C65, C7, C71, C8, C9, JP1, JP10, JP11, JP12, JP13, JP14, JP15, JP16, JP17, JP18, JP20, JP21, JP22, JP23, Q1, Q2, R12, R13, R14, R15, R16, R17, R18, R19, R20, R21, R23, R24, R25, R26, R3, R34, R35, R36, R37, R4, R40, R41, R42, R43, R5, R8, R9, U10, U12, U9: moved to B.Cu
- J1: footprint Connector_IDC:IDC-Header_2x07_P2.54mm_Vertical -> centrifuge footprints:878311411
- U4, U8: footprint Package_QFP:TQFP-100-1EP_14x14mm_P0.5mm_EP5x5mm_ThermalVias -> centrifuge footprints:TQFP-100-1EP_14x14mm_P0.5mm_EP5x5mm_ThermalVias_elprint
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Connections:
- net /pwr_jtag/CONFIG_DONE renamed /CONFIG_DONE
- net /pwr_jtag/PROGRAM_B renamed /PROGRAM_B
- net /vga_interface1/SCL_MCU renamed /SCL_MCU_SL1
- net /vga_interface1/SDA_MCU renamed /SDA_MCU_SL1
- net /vga_interface2/SCL_MCU renamed /SCL_MCU_SL0
- net /vga_interface2/SDA_MCU renamed /SDA_MCU_SL0
- net Net-(J1-Pad10) renamed /pwr_jtag/TDI
- net Net-(J1-Pad8) renamed /pwr_jtag/TDO
- C1 pad 1: +3.3VA -> +3V3
- C1 pad 2: GND -> EP_GND
- C10 pad 1: +1V8 -> +1V9
- C10 pad 2: GND -> EP_GND
- C11 pad 1: +1V8 -> +1V9
- C11 pad 2: GND -> EP_GND
- C12 pad 1: +1V8 -> +1V9
- C12 pad 2: GND -> EP_GND
- C16 pad 1: +1V8 -> +1V9
- C16 pad 2: GND -> EP_GND
- C17 pad 2: GND -> EP_GND
- C18 pad 1: +1V8 -> +1V9
- C18 pad 2: GND -> EP_GND
- C19 pad 2: GND -> EP_GND
- C2 pad 1: +3.3VA -> +3V3
- C2 pad 2: GND -> EP_GND
- C20 pad 1: +1V8 -> +1V9
- C20 pad 2: GND -> EP_GND
- C21 pad 2: GND -> EP_GND
- C22 pad 2: GND -> EP_GND
- C23 pad 1: +3.3VA -> +3V3
- C23 pad 2: GND -> EP_GND
- C24 pad 2: GND -> EP_GND
- C25 pad 2: GND -> EP_GND
- C26 pad 1: +3.3VA -> +3V3
- C26 pad 2: GND -> EP_GND
- C27 pad 2: GND -> EP_GND
- C28 pad 2: GND -> EP_GND
- C29 pad 1: +3.3VA -> +3V3
- C29 pad 2: GND -> EP_GND
- C3 pad 2: GND -> EP_GND
- C30 pad 2: GND -> EP_GND
- C31 pad 1: +3.3VA -> +3V3
- C31 pad 2: GND -> EP_GND
- C32 pad 2: GND -> EP_GND
- C33 pad 2: GND -> EP_GND
- C34 pad 2: GND -> EP_GND
- C35 pad 2: GND -> EP_GND
- C36 pad 2: GND -> EP_GND
- C39 pad 1: +1V8 -> +1V9
- C39 pad 2: GND -> EP_GND
- C4 pad 1: +3.3VA -> +3V3
- C4 pad 2: GND -> EP_GND
- C40 pad 1: +1V8 -> +1V9
- C40 pad 2: GND -> EP_GND
- C41 pad 1: +1V8 -> +1V9
- C41 pad 2: GND -> EP_GND
- C45 pad 1: +1V8 -> +1V9
- C45 pad 2: GND -> EP_GND
- C46 pad 2: GND -> EP_GND
- C47 pad 1: +1V8 -> +1V9
- C47 pad 2: GND -> EP_GND
- C48 pad 2: GND -> EP_GND
- C49 pad 1: +1V8 -> +1V9
- C49 pad 2: GND -> EP_GND
- C5 pad 1: +3.3VA -> +3V3
- C5 pad 2: GND -> EP_GND
- C50 pad 2: GND -> EP_GND
- C51 pad 2: GND -> EP_GND
- C52 pad 1: +3.3VA -> +3V3
- C52 pad 2: GND -> EP_GND
- C53 pad 2: GND -> EP_GND
- C54 pad 2: GND -> EP_GND
- C55 pad 1: +3.3VA -> +3V3
- C55 pad 2: GND -> EP_GND
- C56 pad 2: GND -> EP_GND
- C57 pad 2: GND -> EP_GND
- C58 pad 1: +3.3VA -> +3V3
- C58 pad 2: GND -> EP_GND
- C59 pad 2: GND -> EP_GND
- C6 pad 2: GND -> EP_GND
- C60 pad 1: +3.3VA -> +3V3
- C60 pad 2: GND -> EP_GND
- C61 pad 2: GND -> EP_GND
- C62 pad 2: GND -> EP_GND
- C63 pad 2: GND -> EP_GND
- C64 pad 2: GND -> EP_GND
- C65 pad 2: GND -> EP_GND
- C68 pad 1: +3.3VA -> +3V3
- C68 pad 2: GND -> EP_GND
- C69 pad 1: +3.3VA -> +3V3
- C69 pad 2: GND -> EP_GND
- C7 pad 2: GND -> EP_GND
- C70 pad 1: +3.3VA -> +3V3
- C70 pad 2: GND -> EP_GND
- C71 pad 1: +3.3VA -> +3V3
- C71 pad 2: GND -> EP_GND
- C8 pad 2: GND -> EP_GND
- C9 pad 2: GND -> EP_GND
- J1 pad 1: GND -> EP_GND
- J1 pad 11: GND -> EP_GND
- J1 pad 13: GND -> EP_GND
- J1 pad 2: /pwr_jtag/VREF -> +1V8
- J1 pad 3: GND -> EP_GND
- J1 pad 4: Net-(J1-Pad4) -> /pwr_jtag/TMS
- J1 pad 5: GND -> EP_GND
- J1 pad 6: Net-(J1-Pad6) -> /pwr_jtag/TCK
- J1 pad 7: GND -> EP_GND
- J1 pad 9: GND -> EP_GND
- J2 pad 10: GND -> EP_GND
- J2 pad 5: GND -> EP_GND
- J2 pad 6: GND -> EP_GND
- J2 pad 7: GND -> EP_GND
- J2 pad 8: GND -> EP_GND
- J3 pad 10: GND -> EP_GND
- J3 pad 5: GND -> EP_GND
- J3 pad 6: GND -> EP_GND
- J3 pad 7: GND -> EP_GND
- J3 pad 8: GND -> EP_GND
- J4 pad 10: GND -> EP_GND
- J4 pad 5: GND -> EP_GND
- J4 pad 6: GND -> EP_GND
- J4 pad 7: GND -> EP_GND
- J4 pad 8: GND -> EP_GND
- JP11 pad 1: GND -> EP_GND
- JP12 pad 1: GND -> EP_GND
- JP13 pad 1: GND -> EP_GND
- JP14 pad 1: GND -> EP_GND
- JP18 pad 1: GND -> EP_GND
- JP19 pad 1: GND -> EP_GND
- JP20 pad 1: GND -> EP_GND
- JP21 pad 1: GND -> EP_GND
- Q1 pad 1: +3.3VA -> +3V3
- Q1 pad 2: /vga_interface/SDA_MCU -> /SDA_MCU_MASTER
- Q2 pad 1: +3.3VA -> +3V3
- Q2 pad 2: /vga_interface/SCL_MCU -> /SCL_MCU_MASTER
- Q3 pad 1: +3.3VA -> +3V3
- Q4 pad 1: +3.3VA -> +3V3
- Q5 pad 1: +3.3VA -> +3V3
- Q6 pad 1: +3.3VA -> +3V3
- R1 pad 1: +3.3VA -> +3V3
- R10 pad 1: /pwr_jtag/VCCO_0 -> +3V3
- R11 pad 1: /pwr_jtag/VCCO_0 -> +3V3
- R12 pad 1: +3.3VA -> +3V3
- R12 pad 2: /vga_interface/SDA_MCU -> /SDA_MCU_MASTER
- R13 pad 1: +3.3VA -> +3V3
- R13 pad 2: /vga_interface/SCL_MCU -> /SCL_MCU_MASTER
- R18 pad 1: +3.3VA -> +3V3
- R19 pad 1: +3.3VA -> +3V3
- R2 pad 1: +3.3VA -> +3V3
- R20 pad 1: +3.3VA -> +3V3
- R21 pad 1: +3.3VA -> +3V3
- R23 pad 1: +3.3VA -> +3V3
- R23 pad 2: /vga_input2/SDA -> /SDA_MCU_MASTER
- R24 pad 1: +3.3VA -> +3V3
- R24 pad 2: /vga_input2/SCL -> /SCL_MCU_MASTER
- R25 pad 1: +3.3VA -> +3V3
- R26 pad 2: GND -> EP_GND
- R28 pad 1: +3.3VA -> +3V3
- R28 pad 2: /vga_input1/SDA -> /SDA_MCU_MASTER
- R29 pad 1: +3.3VA -> +3V3
- R29 pad 2: /vga_input1/SCL -> /SCL_MCU_MASTER
- R3 pad 2: GND -> EP_GND
- R30 pad 1: +3.3VA -> +3V3
- R31 pad 2: GND -> EP_GND
- R32 pad 1: +3.3VA -> +3V3
- R33 pad 1: +3.3VA -> +3V3
- R38 pad 1: +3.3VA -> +3V3
- R39 pad 1: +3.3VA -> +3V3
- R4 pad 2: GND -> EP_GND
- R44 pad 1: +3.3VA -> +3V3
- R45 pad 1: +3.3VA -> +3V3
- R46 pad 1: +3.3VA -> +3V3
- R5 pad 2: GND -> EP_GND
- R6 pad 2: GND -> EP_GND
- R8 pad 1: /pwr_jtag/VCCO_0 -> +3V3
- R8 pad 2: Net-(J1-Pad6) -> /pwr_jtag/TMS
- R9 pad 1: /pwr_jtag/VCCO_0 -> +3V3
- R9 pad 2: Net-(J1-Pad4) -> /pwr_jtag/TCK
- U1 pad A1: GND -> EP_GND
- U1 pad A11: GND -> EP_GND
- U1 pad A16: +3.3VA -> +3V3
- U1 pad A2: unconnected-(U1-PadA2) -> /fpga_core/IN0.B5
- U1 pad A3: /fpga_core/IN0.G6 -> /fpga_core/IN0.G8
- U1 pad A4: /fpga_core/IN0.G8 -> /fpga_core/IN0.G7
- U1 pad A5: /fpga_core/IN0.G9 -> /fpga_core/IN0.R9
- U1 pad A6: +3.3VA -> +3V3
- U1 pad A7: /fpga_core/IN0.R7 -> /fpga_core/IN0.R6
- U1 pad A8: unconnected-(U1-PadA8) -> /config_sram/AUXIO15
- U1 pad A9: unconnected-(U1-PadA9) -> /config_sram/AUXIO14
- U1 pad B1: /fpga_core/FIDIN0 -> /fpga_core/IN0.B7
- U1 pad B13: +3.3VA -> +3V3
- U1 pad B2: /fpga_core/IN0.B5 -> /fpga_core/IN0.B6
- U1 pad B3: +3.3VA -> +3V3
- U1 pad B4: /fpga_core/IN0.G7 -> /fpga_core/IN0.G6
- U1 pad B5: /fpga_core/IN0.R5 -> /fpga_core/IN0.R8
- U1 pad B6: /fpga_core/IN0.R6 -> /fpga_core/IN0.R7
- U1 pad B7: /fpga_core/IN0.R8 -> /fpga_core/IN0.R5
- U1 pad B8: GND -> EP_GND
- U1 pad B9: unconnected-(U1-PadB9) -> /config_sram/AUXIO13
- U1 pad C1: unconnected-(U1-PadC1) -> /fpga_core/IN0.B9
- U1 pad C10: +3.3VA -> +3V3
- U1 pad C15: GND -> EP_GND
- U1 pad C2: /fpga_core/IN0.B6 -> /fpga_core/IN0.B8
- U1 pad C3: /fpga_core/IN0.B7 -> /fpga_core/IN0.G9
- U1 pad C4: unconnected-(U1-PadC4) -> /fpga_core/AUXIO18
- U1 pad C5: GND -> EP_GND
- U1 pad C6: /fpga_core/IN0.G4 -> /fpga_core/AUXIO22
- U1 pad C7: /fpga_core/IN0.G5 -> /fpga_core/AUXIO23
- U1 pad C9: unconnected-(U1-PadC9) -> /config_sram/AUXIO16
- U1 pad D1: /fpga_core/VSIN0 -> /fpga_core/HSIN0
- U1 pad D12: GND -> EP_GND
- U1 pad D2: GND -> EP_GND
- U1 pad D3: unconnected-(U1-PadD3) -> /fpga_core/IN0.G4
- U1 pad D4: unconnected-(U1-PadD4) -> /fpga_core/AUXIO19
- U1 pad D5: /fpga_core/IN0.B8 -> /fpga_core/AUXIO20
- U1 pad D6: /fpga_core/IN0.B9 -> /fpga_core/AUXIO21
- U1 pad D7: +3.3VA -> +3V3
- U1 pad E1: /fpga_core/IN1.R8 -> /fpga_core/FIDIN0
- U1 pad E10: unconnected-(U1-PadE10) -> +1V0
- U1 pad E14: +3.3VA -> +3V3
- U1 pad E2: /fpga_core/HSIN0 -> /fpga_core/VSIN0
- U1 pad E3: /fpga_core/DATACLKIN0 -> /fpga_core/IN0.G5
- U1 pad E4: +3.3VA -> +3V3
- U1 pad E5: /fpga_core/HSIN1 -> /fpga_core/DATACLKIN0
- U1 pad E6: /fpga_core/IN0.R9 -> /fpga_core/AUXIO24
- U1 pad E7: unconnected-(U1-PadE7) -> +3V3
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Routing:
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- added copper zone on B.Cu, net +1V0
- added copper zone on In3.Cu, net +1V8
- added copper zone on B.Cu, net +1V9
- added copper zone on In4.Cu, net +3V3
- added copper zone on In1.Cu, net EP_GND
- removed copper zone on In6.Cu, net +3.3VA
- removed copper zone on In1.Cu, net GND
Other:
- board outline added: 184.8 x 96.6 mm
- copper layers 8 -> 6
- board text added: "PROGRAM_B"
- board text added: "VGA Centrifuge R1 Schematics & PCB: Håvard Krogstie, Paolo Celati FPGA Design: Jostein Bakkevig, Erik Martinsen, Eirik Tanberg MCU Programming: Jesper Norsted, Marius Arhaug, Amandus Thorsrud"
