File: centrifuge/vga_output.kicad_sch (KiCad schematic)
At the start: 0 parts

Commit message: Completed majority of schematic, need to add decoupling but otherwise mostly ready
Parts:
- added C1, C2, C7, C8: 10u, Capacitor_SMD:C_0805_2012Metric_Pad1.18x1.45mm_HandSolder, symbol Device:C_Small
- added C3, C4, C5, C6, C9: 0.1u, Capacitor_SMD:C_0805_2012Metric_Pad1.18x1.45mm_HandSolder, symbol Device:C_Small
- added R3, R4, R5: 75, Resistor_SMD:R_0805_2012Metric_Pad1.20x1.40mm_HandSolder, symbol Device:R_Small
- added R6: 3.8k, Resistor_SMD:R_0805_2012Metric_Pad1.20x1.40mm_HandSolder, symbol Device:R_Small
- added R7: 2.2k, Resistor_SMD:R_0805_2012Metric_Pad1.20x1.40mm_HandSolder, symbol Device:R_Small
- added U5: THS8136, Package_QFP:LQFP-48-1EP_7x7mm_P0.5mm_EP3.6x3.6mm, symbol centrifuge_symbols:THS8136
Connections:
- new net +1V8: C7.1, C8.1, C9.1, R7.1, U5.12 (DVDD)
- new net +3V3: C1.1, C2.1, C4.1, C5.1, U5.40 (AVDD), U5.44 (AVDD)
- new net B0: U5.10 (B0), U5.13 (R0), U5.14 (R1), U5.15 (R2), U5.16 (R3), U5.17 (R4), U5.33 (G3), U5.34 (G2), U5.35 (G1), U5.36 (G0), U5.6 (B4), U5.7 (B3), U5.8 (B2), U5.9 (B1)
- new net B5: U5.5 (B5)
- new net B6: U5.4 (B6)
- new net B7: U5.3 (B7)
- new net B8: U5.2 (B8)
- new net B9: U5.1 (B9)
- new net B_OUT: R3.1, U5.45 (AB)
- new net COMP: C3.1, U5.39 (COMP)
- new net DAC_CLK: U5.26 (CLK)
- new net FSADJ: R6.1, U5.38 (FSADJ)
- new net G4: U5.32 (G4)
- new net G5: U5.31 (G5)
- new net G6: U5.30 (G6)
- new net G7: U5.29 (G7)
- new net G8: U5.28 (G8)
- new net G9: U5.27 (G9)
- new net GND: C1.2, C2.2, C3.2, C4.2, C5.2, C6.2, C7.2, C8.2, C9.2, R3.2, R4.2, R5.2, R6.2, U5.11 (DVSS), U5.42 (AVSS), U5.46 (AVSS), U5.47 (M1), U5.48 (M2)
- new net G_OUT: R5.1, U5.41 (AG)
- new net R5: U5.18 (R5)
- new net R6: U5.19 (R6)
- new net R7: U5.20 (R7)
- new net R8: U5.21 (R8)
- new net R9: U5.22 (R9)
- new net R_OUT: R4.1, U5.43 (AR)
- new net SYNC_T: R7.2, U5.23 (~{BLANK}), U5.24 (~{SYNC}), U5.25 (SYNC_T)
- new net VREF: C6.1, U5.37 (VREF)
Other:
- note added: "Going for 5-6-5 bits for R-G-B respectively Rest are sadly grounded"
- note added: "Not using DAC-generated sync"
- note added: "datasheet recommends 3.8k on rfsadj for our 700 mV outputs"
- title: (none) -> VGA Centrifuge

Commit message: FPGA PCB design completed
Connections:
- net B0 is gone; now on net GND: U5.10 (B0), U5.13 (R0), U5.14 (R1), U5.15 (R2), U5.16 (R3), U5.17 (R4), U5.33 (G3), U5.34 (G2), U5.35 (G1), U5.36 (G0), U5.6 (B4), U5.7 (B3), U5.8 (B2), U5.9 (B1)
Changed lines of the file:
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@@
   (title_block
     (title "VGA Centrifuge")
+    (date "2022-09-30")
     (rev "R1")
     (comment 1 "Author: Paolo Celati")
+    (comment 2 "VGA DAC")
   )
   (junction (at 59.69 99.695) (diameter 0) (color 0 0 0 0)
@@
   (junction (at 160.02 123.19) (diameter 0) (color 0 0 0 0)
   )
+  (junction (at 59.69 108.585) (diameter 0) (color 0 0 0 0)
+  )
   (junction (at 136.525 137.16) (diameter 0) (color 0 0 0 0)
   )
@@
     (stroke (width 0) (type default) (color 0 0 0 0))
   )
+  (wire (pts (xy 59.69 108.585) (xy 59.69 111.125))
+    (stroke (width 0) (type default) (color 0 0 0 0))
+  )
   (bus (pts (xy 62.23 89.535) (xy 62.23 86.995))
     (stroke (width 0) (type default) (color 0 0 0 0))
@@
   )
   (text "datasheet recommends 3.8k on rfsadj\nfor our 700 mV outputs"
-    (at 170.815 164.465 0)
+    (at 146.304 165.989 0)
     (effects (font (size 1.27 1.27)) (justify left bottom))
   )
@@
     (pin "2")
   )
+  (symbol (lib_id "power:GND") (at 59.69 111.125 0) (unit 1)
+    (in_bom yes) (on_board yes) (fields_autoplaced)
+    (property "Reference" "#PWR0216" (id 0) (at 59.69 117.475 0)
+      (effects (font (size 1.27 1.27)) hide)
+    )
+    (property "Value" "GND" (id 1) (at 59.69 115.57 0))
+    (property "Footprint" "" (id 2) (at 59.69 111.125 0)
+      (effects (font (size 1.27 1.27)) hide)
+    )
+    (property "Datasheet" "" (id 3) (at 59.69 111.125 0)
+      (effects (font (size 1.27 1.27)) hide)
+    )
+    (pin "1")
+  )
   (symbol (lib_id "power:GND") (at 221.615 46.99 0) (unit 1)
