File: centrifuge_mcu/centrifuge_mcu.kicad_sch (KiCad schematic)
At the start: 16 parts, among them J101 Conn_02x06_Odd_Even, J102 FPGA_Power, J103 FPGA_extra, J104 FPGA_control, J105 FPGA_SPI, J106 DDC_I2Cs, J107 ACD_I2C, J108 ACD_RST, U101 DFR0555, U102 LCD16x2L

Commit message: slowly but surely decopling and connecting everything to the MCU
Parts:
- J107: value ACD_I2C -> ADC_I2C
- J108: value ACD_RST -> ADC_RST
Connections:
- net +1V0: now also J101.6 (Pin_6), J102.4 (Pin_4); no longer J101.2 (Pin_2), J102.6 (Pin_6)
- net +1V8: now also J101.8 (Pin_8), J102.3 (Pin_3); no longer J101.4 (Pin_4), J102.5 (Pin_5)
- net +1V9: now also J101.4 (Pin_4), J102.5 (Pin_5); no longer J101.8 (Pin_8), J102.3 (Pin_3)
- net +3.3V: now also J101.10 (Pin_10), J102.2 (Pin_2); no longer J101.6 (Pin_6), J102.4 (Pin_4)
- net +3.3VADC: now also J101.2 (Pin_2), J102.6 (Pin_6); no longer J101.10 (Pin_10), J102.2 (Pin_2)
- net Power Circuit/1V0: now also J101.5 (Pin_5); no longer J101.1 (Pin_1)
- net Power Circuit/1V8: now also J101.7 (Pin_7); no longer J101.3 (Pin_3)
- net Power Circuit/1V9: now also J101.3 (Pin_3); no longer J101.7 (Pin_7)
- net Power Circuit/3V3: now also J101.9 (Pin_9); no longer J101.5 (Pin_5)
- net Power Circuit/3V3ADC: now also J101.1 (Pin_1); no longer J101.9 (Pin_9)
