File: centrifuge_combined/mcu_part/SD_card.kicad_sch (KiCad schematic)
At the start: 7 parts

Commit message: Board appears ok
Other:
- title: (none) -> VGA Centrifuge
Changed lines of the file:
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@@
 (kicad_sch (version 20211123) (generator eeschema)
   (paper "A4")
+  (title_block
+    (title "VGA Centrifuge")
+    (date "2022-10-03")
+    (rev "R2")
+  )
   (junction (at 149.86 81.28) (diameter 0) (color 0 0 0 0)
   )

Commit message: fixed keypad hole sizes, and submitted
Parts:
- C535: value (none) -> 100n
- J513: value (none) -> SD_Card
- R523, R524, R525, R526, R527: value (none) -> 10k
Changed lines of the file:
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@@
       (effects (font (size 1.27 1.27)) hide)
     )
-    (property "Value" "" (id 1) (at 140.97 91.44 0))
+    (property "Value" "GND" (id 1) (at 140.97 91.44 0))
     (property "Footprint" "" (id 2) (at 140.97 86.36 0)
       (effects (font (size 1.27 1.27)) hide)
@@
       (effects (font (size 1.27 1.27)) (justify left))
     )
-    (property "Value" "" (id 1) (at 139.7 59.69 90)
+    (property "Value" "10k" (id 1) (at 139.7 59.69 90)
       (effects (font (size 1.27 1.27)) (justify left))
     )
@@
       (effects (font (size 1.27 1.27)) (justify left))
     )
-    (property "Value" "" (id 1) (at 147.955 92.075 0)
+    (property "Value" "100n" (id 1) (at 147.955 92.075 0)
       (effects (font (size 1.27 1.27)) (justify left))
     )
@@
     (in_bom yes) (on_board yes) (fields_autoplaced)
     (property "Reference" "J513" (id 0) (at 178.435 58.42 0))
-    (property "Value" "" (id 1) (at 178.435 60.96 0))
+    (property "Value" "SD_Card" (id 1) (at 178.435 60.96 0))
     (property "Footprint" "" (id 2) (at 178.435 76.2 0)
       (effects (font (size 1.27 1.27)) hide)
@@
       (effects (font (size 1.27 1.27)) (justify left))
     )
-    (property "Value" "" (id 1) (at 144.78 59.69 90)
+    (property "Value" "10k" (id 1) (at 144.78 59.69 90)
       (effects (font (size 1.27 1.27)) (justify left))
     )
@@
       (effects (font (size 1.27 1.27)) (justify left))
     )
-    (property "Value" "" (id 1) (at 134.62 55.88 90)
+    (property "Value" "10k" (id 1) (at 134.62 55.88 90)
       (effects (font (size 1.27 1.27)) (justify left))
     )
@@
       (effects (font (size 1.27 1.27)) (justify left))
     )
-    (property "Value" "" (id 1) (at 149.86 59.69 90)
+    (property "Value" "10k" (id 1) (at 149.86 59.69 90)
       (effects (font (size 1.27 1.27)) (justify left))
     )
@@
       (effects (font (size 1.27 1.27)) (justify left))
     )
-    (property "Value" "" (id 1) (at 155.575 91.44 90)
+    (property "Value" "10k" (id 1) (at 155.575 91.44 90)
       (effects (font (size 1.27 1.27)) (justify left))
     )

Commit message: Fixed missing footprints, added decoupling capacitors, adjusted board edges
Parts:
- C535: footprint (none) -> Capacitor_SMD:C_0805_2012Metric_Pad1.18x1.45mm_HandSolder
- J513: footprint (none) -> Connector_Card:SD_Kyocera_145638009511859+
- R523, R524, R525, R526, R527: footprint (none) -> Resistor_SMD:R_0805_2012Metric_Pad1.20x1.40mm_HandSolder
Changed lines of the file:
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@@
     (title "VGA Centrifuge")
     (date "2022-10-03")
-    (rev "R2")
+    (rev "R3")
+    (comment 1 "Author: Håvard Krogstie")
+    (comment 2 "SD card reader")
   )
   (junction (at 149.86 81.28) (diameter 0) (color 0 0 0 0)
@@
       (effects (font (size 1.27 1.27)) (justify left))
     )
-    (property "Footprint" "" (id 2) (at 137.922 58.42 90)
+    (property "Footprint" "Resistor_SMD:R_0805_2012Metric_Pad1.20x1.40mm_HandSolder" (id 2) (at 137.922 58.42 90)
       (effects (font (size 1.27 1.27)) hide)
     )
@@
       (effects (font (size 1.27 1.27)) (justify left))
     )
-    (property "Footprint" "" (id 2) (at 148.2852 93.98 0)
+    (property "Footprint" "Capacitor_SMD:C_0805_2012Metric_Pad1.18x1.45mm_HandSolder" (id 2) (at 148.2852 93.98 0)
       (effects (font (size 1.27 1.27)) hide)
     )
@@
     (property "Reference" "J513" (id 0) (at 178.435 58.42 0))
     (property "Value" "SD_Card" (id 1) (at 178.435 60.96 0))
-    (property "Footprint" "" (id 2) (at 178.435 76.2 0)
+    (property "Footprint" "Connector_Card:SD_Kyocera_145638009511859+" (id 2) (at 178.435 76.2 0)
       (effects (font (size 1.27 1.27)) hide)
     )
@@
       (effects (font (size 1.27 1.27)) (justify left))
     )
-    (property "Footprint" "" (id 2) (at 143.002 58.42 90)
+    (property "Footprint" "Resistor_SMD:R_0805_2012Metric_Pad1.20x1.40mm_HandSolder" (id 2) (at 143.002 58.42 90)
       (effects (font (size 1.27 1.27)) hide)
     )
@@
       (effects (font (size 1.27 1.27)) (justify left))
     )
-    (property "Footprint" "" (id 2) (at 136.398 58.42 90)
+    (property "Footprint" "Resistor_SMD:R_0805_2012Metric_Pad1.20x1.40mm_HandSolder" (id 2) (at 136.398 58.42 90)
       (effects (font (size 1.27 1.27)) hide)
     )
@@
       (effects (font (size 1.27 1.27)) (justify left))
     )
-    (property "Footprint" "" (id 2) (at 148.082 58.42 90)
+    (property "Footprint" "Resistor_SMD:R_0805_2012Metric_Pad1.20x1.40mm_HandSolder" (id 2) (at 148.082 58.42 90)
       (effects (font (size 1.27 1.27)) hide)
     )
@@
       (effects (font (size 1.27 1.27)) (justify left))
     )
-    (property "Footprint" "" (id 2) (at 153.797 90.17 90)
-      (effects (font (size 1.27 1.27)) hide)
-    )
+    (property "Footprint" "Resistor_SMD:R_0805_2012Metric_Pad1.20x1.40mm_HandSolder" (id 2) (at 153.797 90.17 90)
+      (effects (font (size 1.27 1.27)) hide)
+    )

Commit message: remove digikey links to products that we already buy from mouser, add mouser link instead
Parts:
- R523, R524, R525, R526, R527: Order Page (none) -> https://no.mouser.com/ProductDetail/YAGEO/RC0805FR-1310KL?q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; Purchase https://www.digikey.no/no/products/detail/yageo/AC0805FR-07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 -> (none)
Changed lines of the file:
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@@
       (effects (font (size 1.27 1.27)) hide)
     )
-    (property "Purchase" "https://www.digikey.no/no/products/detail/yageo/AC0805FR-0710KL/2827834" (id 4) (at 139.7 58.42 0)
+    (property "Purchase" "" (id 4) (at 139.7 58.42 0)
+      (effects (font (size 1.27 1.27)) hide)
+    )
+    (property "Order Page" "https://no.mouser.com/ProductDetail/YAGEO/RC0805FR-1310KL?qs=sGAEpiMZZMtlubZbdhIBIHucEnbnlIRRGobQQ23C9vc%3D" (id 5) (at 139.7 58.42 0)
       (effects (font (size 1.27 1.27)) hide)
     )
@@
       (effects (font (size 1.27 1.27)) hide)
     )
-    (property "Purchase" "https://www.digikey.no/no/products/detail/yageo/AC0805FR-0710KL/2827834" (id 4) (at 144.78 58.42 0)
+    (property "Purchase" "" (id 4) (at 144.78 58.42 0)
+      (effects (font (size 1.27 1.27)) hide)
+    )
+    (property "Order Page" "https://no.mouser.com/ProductDetail/YAGEO/RC0805FR-1310KL?qs=sGAEpiMZZMtlubZbdhIBIHucEnbnlIRRGobQQ23C9vc%3D" (id 5) (at 144.78 58.42 0)
       (effects (font (size 1.27 1.27)) hide)
     )
@@
       (effects (font (size 1.27 1.27)) hide)
     )
-    (property "Purchase" "https://www.digikey.no/no/products/detail/yageo/AC0805FR-0710KL/2827834" (id 4) (at 134.62 58.42 0)
+    (property "Purchase" "" (id 4) (at 134.62 58.42 0)
+      (effects (font (size 1.27 1.27)) hide)
+    )
+    (property "Order Page" "https://no.mouser.com/ProductDetail/YAGEO/RC0805FR-1310KL?qs=sGAEpiMZZMtlubZbdhIBIHucEnbnlIRRGobQQ23C9vc%3D" (id 5) (at 134.62 58.42 0)
       (effects (font (size 1.27 1.27)) hide)
     )
@@
       (effects (font (size 1.27 1.27)) hide)
     )
-    (property "Purchase" "https://www.digikey.no/no/products/detail/yageo/AC0805FR-0710KL/2827834" (id 4) (at 149.86 58.42 0)
+    (property "Purchase" "" (id 4) (at 149.86 58.42 0)
+      (effects (font (size 1.27 1.27)) hide)
+    )
+    (property "Order Page" "https://no.mouser.com/ProductDetail/YAGEO/RC0805FR-1310KL?qs=sGAEpiMZZMtlubZbdhIBIHucEnbnlIRRGobQQ23C9vc%3D" (id 5) (at 149.86 58.42 0)
       (effects (font (size 1.27 1.27)) hide)
     )
@@
       (effects (font (size 1.27 1.27)) hide)
     )
-    (property "Purchase" "https://www.digikey.no/no/products/detail/yageo/AC0805FR-0710KL/2827834" (id 4) (at 155.575 90.17 0)
+    (property "Purchase" "" (id 4) (at 155.575 90.17 0)
       (effects (font (size 1.27 1.27)) hide)
     )
+    (property "Order Page" "https://no.mouser.com/ProductDetail/YAGEO/RC0805FR-1310KL?qs=sGAEpiMZZMtlubZbdhIBIHucEnbnlIRRGobQQ23C9vc%3D" (id 5) (at 155.575 90.17 0)
+      (effects (font (size 1.27 1.27)) hide)
+    )

Commit message: Fixed Elprint complaints and JTAG VREF problems+config flash CS
Parts:
- R523, R524, R525, R526, R527: Order Page https://no.mouser.com/ProductDetail/YAGEO/RC0805FR-1310KL?q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 -> (none); Purchase (none) -> https://www.digikey.no/no/products/detail/yageo/AC0805FR-07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
Changed lines of the file:
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@@
   (title_block
     (title "VGA Centrifuge")
-    (date "2022-10-03")
-    (rev "R3")
+    (date "2022-10-05")
+    (rev "R4")
     (comment 1 "Author: Håvard Krogstie")
     (comment 2 "SD card reader")
@@
       (effects (font (size 1.27 1.27)) hide)
     )
-    (property "Purchase" "" (id 4) (at 139.7 58.42 0)
-      (effects (font (size 1.27 1.27)) hide)
-    )
-    (property "Order Page" "https://no.mouser.com/ProductDetail/YAGEO/RC0805FR-1310KL?qs=sGAEpiMZZMtlubZbdhIBIHucEnbnlIRRGobQQ23C9vc%3D" (id 5) (at 139.7 58.42 0)
+    (property "Purchase" "https://www.digikey.no/no/products/detail/yageo/AC0805FR-0710KL/2827834" (id 4) (at 139.7 58.42 0)
       (effects (font (size 1.27 1.27)) hide)
     )
@@
       (effects (font (size 1.27 1.27)) hide)
     )
-    (property "Purchase" "" (id 4) (at 144.78 58.42 0)
-      (effects (font (size 1.27 1.27)) hide)
-    )
-    (property "Order Page" "https://no.mouser.com/ProductDetail/YAGEO/RC0805FR-1310KL?qs=sGAEpiMZZMtlubZbdhIBIHucEnbnlIRRGobQQ23C9vc%3D" (id 5) (at 144.78 58.42 0)
+    (property "Purchase" "https://www.digikey.no/no/products/detail/yageo/AC0805FR-0710KL/2827834" (id 4) (at 144.78 58.42 0)
       (effects (font (size 1.27 1.27)) hide)
     )
@@
       (effects (font (size 1.27 1.27)) hide)
     )
-    (property "Purchase" "" (id 4) (at 134.62 58.42 0)
-      (effects (font (size 1.27 1.27)) hide)
-    )
-    (property "Order Page" "https://no.mouser.com/ProductDetail/YAGEO/RC0805FR-1310KL?qs=sGAEpiMZZMtlubZbdhIBIHucEnbnlIRRGobQQ23C9vc%3D" (id 5) (at 134.62 58.42 0)
+    (property "Purchase" "https://www.digikey.no/no/products/detail/yageo/AC0805FR-0710KL/2827834" (id 4) (at 134.62 58.42 0)
       (effects (font (size 1.27 1.27)) hide)
     )
@@
       (effects (font (size 1.27 1.27)) hide)
     )
-    (property "Purchase" "" (id 4) (at 149.86 58.42 0)
-      (effects (font (size 1.27 1.27)) hide)
-    )
-    (property "Order Page" "https://no.mouser.com/ProductDetail/YAGEO/RC0805FR-1310KL?qs=sGAEpiMZZMtlubZbdhIBIHucEnbnlIRRGobQQ23C9vc%3D" (id 5) (at 149.86 58.42 0)
+    (property "Purchase" "https://www.digikey.no/no/products/detail/yageo/AC0805FR-0710KL/2827834" (id 4) (at 149.86 58.42 0)
       (effects (font (size 1.27 1.27)) hide)
     )
@@
       (effects (font (size 1.27 1.27)) hide)
     )
-    (property "Purchase" "" (id 4) (at 155.575 90.17 0)
-      (effects (font (size 1.27 1.27)) hide)
-    )
-    (property "Order Page" "https://no.mouser.com/ProductDetail/YAGEO/RC0805FR-1310KL?qs=sGAEpiMZZMtlubZbdhIBIHucEnbnlIRRGobQQ23C9vc%3D" (id 5) (at 155.575 90.17 0)
-      (effects (font (size 1.27 1.27)) hide)
-    )
+    (property "Purchase" "https://www.digikey.no/no/products/detail/yageo/AC0805FR-0710KL/2827834" (id 4) (at 155.575 90.17 0)
+      (effects (font (size 1.27 1.27)) hide)
+    )
