File: centrifuge_combined/mcu_part/button_panel.kicad_sch (KiCad schematic)
At the start: 5 parts

Commit message: Board appears ok
Other:
- title: (none) -> VGA Centrifuge
Changed lines of the file:
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@@
 (kicad_sch (version 20211123) (generator eeschema)
   (paper "A4")
+  (title_block
+    (title "VGA Centrifuge")
+    (date "2022-10-03")
+    (rev "R2")
+  )
   (wire (pts (xy 170.18 125.73) (xy 180.975 125.73))
     (stroke (width 0) (type default) (color 0 0 0 0))

Commit message: fixed keypad hole sizes, and submitted
Parts:
- R529, R530, R531, R532: value (none) -> 10k
- U507: value (none) -> 4x4_keyboard
Changed lines of the file:
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@@
       (effects (font (size 1.27 1.27)) (justify left))
     )
-    (property "Value" "" (id 1) (at 167.64 85.7249 0)
+    (property "Value" "4x4_keyboard" (id 1) (at 167.64 85.7249 0)
       (effects (font (size 1.27 1.27)) (justify left))
     )
@@
     (in_bom yes) (on_board yes)
     (property "Reference" "R529" (id 0) (at 166.37 115.57 90))
-    (property "Value" "" (id 1) (at 166.37 118.11 90))
+    (property "Value" "10k" (id 1) (at 166.37 118.11 90))
     (property "Footprint" "" (id 2) (at 166.37 119.888 90)
       (effects (font (size 1.27 1.27)) hide)
@@
     (in_bom yes) (on_board yes)
     (property "Reference" "R531" (id 0) (at 173.99 111.76 90))
-    (property "Value" "" (id 1) (at 173.99 114.3 90))
+    (property "Value" "10k" (id 1) (at 173.99 114.3 90))
     (property "Footprint" "" (id 2) (at 173.99 116.078 90)
       (effects (font (size 1.27 1.27)) hide)
@@
     (in_bom yes) (on_board yes)
     (property "Reference" "R532" (id 0) (at 173.99 119.38 90))
-    (property "Value" "" (id 1) (at 173.99 121.92 90))
+    (property "Value" "10k" (id 1) (at 173.99 121.92 90))
     (property "Footprint" "" (id 2) (at 173.99 123.698 90)
       (effects (font (size 1.27 1.27)) hide)
@@
     (in_bom yes) (on_board yes)
     (property "Reference" "R530" (id 0) (at 166.37 123.19 90))
-    (property "Value" "" (id 1) (at 166.37 125.73 90))
+    (property "Value" "10k" (id 1) (at 166.37 125.73 90))
     (property "Footprint" "" (id 2) (at 166.37 127.508 90)
       (effects (font (size 1.27 1.27)) hide)

Commit message: Fixed missing footprints, added decoupling capacitors, adjusted board edges
Parts:
- R529, R530, R531, R532: footprint (none) -> Resistor_SMD:R_0805_2012Metric_Pad1.20x1.40mm_HandSolder
- U507: footprint (none) -> centrifuge_mcu:Adafruit 3844
Changed lines of the file:
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@@
     (title "VGA Centrifuge")
     (date "2022-10-03")
-    (rev "R2")
+    (rev "R3")
+    (comment 1 "Author: Håvard Krogstie")
+    (comment 2 "Keypad")
   )
   (wire (pts (xy 170.18 125.73) (xy 180.975 125.73))
@@
       (effects (font (size 1.27 1.27)) (justify left))
     )
-    (property "Footprint" "" (id 2) (at 153.67 91.44 0)
+    (property "Footprint" "centrifuge_mcu:Adafruit 3844" (id 2) (at 153.67 91.44 0)
       (effects (font (size 1.27 1.27)) hide)
     )
@@
     (property "Reference" "R529" (id 0) (at 166.37 115.57 90))
     (property "Value" "10k" (id 1) (at 166.37 118.11 90))
-    (property "Footprint" "" (id 2) (at 166.37 119.888 90)
+    (property "Footprint" "Resistor_SMD:R_0805_2012Metric_Pad1.20x1.40mm_HandSolder" (id 2) (at 166.37 119.888 90)
       (effects (font (size 1.27 1.27)) hide)
     )
@@
     (property "Reference" "R531" (id 0) (at 173.99 111.76 90))
     (property "Value" "10k" (id 1) (at 173.99 114.3 90))
-    (property "Footprint" "" (id 2) (at 173.99 116.078 90)
+    (property "Footprint" "Resistor_SMD:R_0805_2012Metric_Pad1.20x1.40mm_HandSolder" (id 2) (at 173.99 116.078 90)
       (effects (font (size 1.27 1.27)) hide)
     )
@@
     (property "Reference" "R532" (id 0) (at 173.99 119.38 90))
     (property "Value" "10k" (id 1) (at 173.99 121.92 90))
-    (property "Footprint" "" (id 2) (at 173.99 123.698 90)
+    (property "Footprint" "Resistor_SMD:R_0805_2012Metric_Pad1.20x1.40mm_HandSolder" (id 2) (at 173.99 123.698 90)
       (effects (font (size 1.27 1.27)) hide)
     )
@@
     (property "Reference" "R530" (id 0) (at 166.37 123.19 90))
     (property "Value" "10k" (id 1) (at 166.37 125.73 90))
-    (property "Footprint" "" (id 2) (at 166.37 127.508 90)
+    (property "Footprint" "Resistor_SMD:R_0805_2012Metric_Pad1.20x1.40mm_HandSolder" (id 2) (at 166.37 127.508 90)
       (effects (font (size 1.27 1.27)) hide)
     )

Commit message: remove digikey links to products that we already buy from mouser, add mouser link instead
Parts:
- R529, R530, R531, R532: Order Page (none) -> https://no.mouser.com/ProductDetail/YAGEO/RC0805FR-1310KL?q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; Purchase https://www.digikey.no/no/products/detail/yageo/AC0805FR-07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 -> (none)
Changed lines of the file:
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@@
       (effects (font (size 1.27 1.27)) hide)
     )
-    (property "Purchase" "https://www.digikey.no/no/products/detail/yageo/AC0805FR-0710KL/2827834" (id 4) (at 166.37 118.11 0)
+    (property "Purchase" "" (id 4) (at 166.37 118.11 0)
+      (effects (font (size 1.27 1.27)) hide)
+    )
+    (property "Order Page" "https://no.mouser.com/ProductDetail/YAGEO/RC0805FR-1310KL?qs=sGAEpiMZZMtlubZbdhIBIHucEnbnlIRRGobQQ23C9vc%3D" (id 5) (at 166.37 118.11 0)
       (effects (font (size 1.27 1.27)) hide)
     )
@@
       (effects (font (size 1.27 1.27)) hide)
     )
-    (property "Purchase" "https://www.digikey.no/no/products/detail/yageo/AC0805FR-0710KL/2827834" (id 4) (at 173.99 114.3 0)
+    (property "Purchase" "" (id 4) (at 173.99 114.3 0)
+      (effects (font (size 1.27 1.27)) hide)
+    )
+    (property "Order Page" "https://no.mouser.com/ProductDetail/YAGEO/RC0805FR-1310KL?qs=sGAEpiMZZMtlubZbdhIBIHucEnbnlIRRGobQQ23C9vc%3D" (id 5) (at 173.99 114.3 0)
       (effects (font (size 1.27 1.27)) hide)
     )
@@
       (effects (font (size 1.27 1.27)) hide)
     )
-    (property "Purchase" "https://www.digikey.no/no/products/detail/yageo/AC0805FR-0710KL/2827834" (id 4) (at 173.99 121.92 0)
+    (property "Purchase" "" (id 4) (at 173.99 121.92 0)
+      (effects (font (size 1.27 1.27)) hide)
+    )
+    (property "Order Page" "https://no.mouser.com/ProductDetail/YAGEO/RC0805FR-1310KL?qs=sGAEpiMZZMtlubZbdhIBIHucEnbnlIRRGobQQ23C9vc%3D" (id 5) (at 173.99 121.92 0)
       (effects (font (size 1.27 1.27)) hide)
     )
@@
       (effects (font (size 1.27 1.27)) hide)
     )
-    (property "Purchase" "https://www.digikey.no/no/products/detail/yageo/AC0805FR-0710KL/2827834" (id 4) (at 166.37 125.73 0)
+    (property "Purchase" "" (id 4) (at 166.37 125.73 0)
       (effects (font (size 1.27 1.27)) hide)
     )
+    (property "Order Page" "https://no.mouser.com/ProductDetail/YAGEO/RC0805FR-1310KL?qs=sGAEpiMZZMtlubZbdhIBIHucEnbnlIRRGobQQ23C9vc%3D" (id 5) (at 166.37 125.73 0)
+      (effects (font (size 1.27 1.27)) hide)
+    )

Commit message: Fixed Elprint complaints and JTAG VREF problems+config flash CS
Parts:
- R529, R530, R531, R532: Order Page https://no.mouser.com/ProductDetail/YAGEO/RC0805FR-1310KL?q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 -> (none); Purchase (none) -> https://www.digikey.no/no/products/detail/yageo/AC0805FR-07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
Changed lines of the file:
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@@
   (title_block
     (title "VGA Centrifuge")
-    (date "2022-10-03")
-    (rev "R3")
+    (date "2022-10-05")
+    (rev "R4")
     (comment 1 "Author: Håvard Krogstie")
     (comment 2 "Keypad")
@@
       (effects (font (size 1.27 1.27)) hide)
     )
-    (property "Purchase" "" (id 4) (at 166.37 118.11 0)
-      (effects (font (size 1.27 1.27)) hide)
-    )
-    (property "Order Page" "https://no.mouser.com/ProductDetail/YAGEO/RC0805FR-1310KL?qs=sGAEpiMZZMtlubZbdhIBIHucEnbnlIRRGobQQ23C9vc%3D" (id 5) (at 166.37 118.11 0)
+    (property "Purchase" "https://www.digikey.no/no/products/detail/yageo/AC0805FR-0710KL/2827834" (id 4) (at 166.37 118.11 0)
       (effects (font (size 1.27 1.27)) hide)
     )
@@
       (effects (font (size 1.27 1.27)) hide)
     )
-    (property "Purchase" "" (id 4) (at 173.99 114.3 0)
-      (effects (font (size 1.27 1.27)) hide)
-    )
-    (property "Order Page" "https://no.mouser.com/ProductDetail/YAGEO/RC0805FR-1310KL?qs=sGAEpiMZZMtlubZbdhIBIHucEnbnlIRRGobQQ23C9vc%3D" (id 5) (at 173.99 114.3 0)
+    (property "Purchase" "https://www.digikey.no/no/products/detail/yageo/AC0805FR-0710KL/2827834" (id 4) (at 173.99 114.3 0)
       (effects (font (size 1.27 1.27)) hide)
     )
@@
       (effects (font (size 1.27 1.27)) hide)
     )
-    (property "Purchase" "" (id 4) (at 173.99 121.92 0)
-      (effects (font (size 1.27 1.27)) hide)
-    )
-    (property "Order Page" "https://no.mouser.com/ProductDetail/YAGEO/RC0805FR-1310KL?qs=sGAEpiMZZMtlubZbdhIBIHucEnbnlIRRGobQQ23C9vc%3D" (id 5) (at 173.99 121.92 0)
+    (property "Purchase" "https://www.digikey.no/no/products/detail/yageo/AC0805FR-0710KL/2827834" (id 4) (at 173.99 121.92 0)
       (effects (font (size 1.27 1.27)) hide)
     )
@@
       (effects (font (size 1.27 1.27)) hide)
     )
-    (property "Purchase" "" (id 4) (at 166.37 125.73 0)
+    (property "Purchase" "https://www.digikey.no/no/products/detail/yageo/AC0805FR-0710KL/2827834" (id 4) (at 166.37 125.73 0)
       (effects (font (size 1.27 1.27)) hide)
     )
-    (property "Order Page" "https://no.mouser.com/ProductDetail/YAGEO/RC0805FR-1310KL?qs=sGAEpiMZZMtlubZbdhIBIHucEnbnlIRRGobQQ23C9vc%3D" (id 5) (at 166.37 125.73 0)
-      (effects (font (size 1.27 1.27)) hide)
-    )
