File: centrifuge_combined/mcu_part/centrifuge_mcu.kicad_sch (KiCad schematic)
At the start: 17 parts, among them J516 Conn_02x06_Odd_Even

Commit message: Almost finished releasable version
Parts:
- removed J502: (no value), symbol Connector:Conn_01x06_Male
- removed J504, J506: (no value), symbol Connector:Conn_01x04_Male
- added J506: DDCI2C2, Connector_PinHeader_2.54mm:PinHeader_1x02_P2.54mm_Vertical, symbol Connector:Conn_01x02_Male
- added J517: DDCI2C1, Connector_PinHeader_2.54mm:PinHeader_1x02_P2.54mm_Vertical, symbol Connector:Conn_01x02_Male
Connections:
- net I2C0_SCL#1: now also J517.2 (Pin_2)
- net I2C0_SCL#2: now also J506.2 (Pin_2)
- net I2C0_SDA#1: now also J517.1 (Pin_1)
- net I2C0_SDA#2: now also J506.1 (Pin_1)

Commit message: Board appears ok
Connections:
- net +1V8_FPGA: now also J501.2 (Pin_2); no longer J501.8 (Pin_8)
- net +1V9_FPGA: now also J501.8 (Pin_8); no longer J501.4 (Pin_4)
- net +3V3A_FPGA: now also J501.12 (Pin_12); no longer J501.2 (Pin_2)
- net +3V3_FPGA: now also J501.4 (Pin_4); no longer J501.10 (Pin_10)
- net +3V3_MCU: now also J516.4 (Pin_4); no longer J516.10 (Pin_10)
- net +5V_FPGA: now also J501.10 (Pin_10); no longer J501.12 (Pin_12)
- net Power Circuit/1V8: now also J501.1 (Pin_1), J516.1 (Pin_1), J516.2 (Pin_2); no longer J501.7 (Pin_7), J516.7 (Pin_7), J516.8 (Pin_8)
- net Power Circuit/1V9: now also J501.7 (Pin_7), J516.7 (Pin_7), J516.8 (Pin_8); no longer J501.3 (Pin_3), J516.3 (Pin_3), J516.4 (Pin_4)
- net Power Circuit/3V3: now also J501.3 (Pin_3), J516.3 (Pin_3); no longer J501.9 (Pin_9), J516.9 (Pin_9)
- net Power Circuit/3V3ADC: now also J501.11 (Pin_11), J516.11 (Pin_11), J516.12 (Pin_12); no longer J501.1 (Pin_1), J516.1 (Pin_1), J516.2 (Pin_2)
- net Power Circuit/5V0: now also J501.9 (Pin_9), J516.10 (Pin_10), J516.9 (Pin_9); no longer J501.11 (Pin_11), J516.11 (Pin_11), J516.12 (Pin_12)
Other:
- title: VGA Centrifuge - MCU area -> VGA Centrifuge
Changed lines of the file:
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@@
   (paper "A4")
   (title_block
-    (title "VGA Centrifuge - MCU area")
-    (rev "v01")
+    (title "VGA Centrifuge")
+    (date "2022-10-03")
+    (rev "R2")
   )
   (junction (at 71.755 60.325) (diameter 0) (color 0 0 0 0)
@@
   (junction (at 76.835 66.675) (diameter 0) (color 0 0 0 0)
   )
-  (junction (at 41.402 92.329) (diameter 0) (color 0 0 0 0)
-  )
   (junction (at 189.865 70.485) (diameter 0) (color 0 0 0 0)
   )
@@
   (junction (at 136.525 40.386) (diameter 0) (color 0 0 0 0)
   )
+  (junction (at 49.022 92.329) (diameter 0) (color 0 0 0 0)
+  )
   (junction (at 168.275 46.99) (diameter 0) (color 0 0 0 0)
   )
@@
     (stroke (width 0) (type default) (color 0 0 0 0))
   )
+  (wire (pts (xy 49.022 79.629) (xy 49.022 92.329))
+    (stroke (width 0) (type default) (color 0 0 0 0))
+  )
   (wire (pts (xy 196.85 29.845) (xy 196.85 51.054))
     (stroke (width 0) (type default) (color 0 0 0 0))
@@
     (stroke (width 0) (type default) (color 0 0 0 0))
   )
-  (wire (pts (xy 41.402 79.629) (xy 41.402 92.329))
-    (stroke (width 0) (type default) (color 0 0 0 0))
-  )
   (wire (pts (xy 71.755 60.325) (xy 71.755 82.423))
     (stroke (width 0) (type default) (color 0 0 0 0))
@@
     (stroke (width 0) (type default) (color 0 0 0 0))
   )
+  (wire (pts (xy 202.057 46.482) (xy 187.325 46.482))
+    (stroke (width 0) (type default) (color 0 0 0 0))
+  )
+  (wire (pts (xy 117.348 54.102) (xy 122.555 54.102))
+    (stroke (width 0) (type default) (color 0 0 0 0))
+  )
+  (wire (pts (xy 148.59 52.197) (xy 148.59 61.595))
+    (stroke (width 0) (type default) (color 0 0 0 0))
+  )
+  (wire (pts (xy 156.21 42.545) (xy 156.21 58.039))
+    (stroke (width 0) (type default) (color 0 0 0 0))
+  )
+  (wire (pts (xy 122.555 54.102) (xy 122.555 61.595))
+    (stroke (width 0) (type default) (color 0 0 0 0))
+  )
+  (wire (pts (xy 196.85 51.054) (xy 196.85 76.2))
+    (stroke (width 0) (type default) (color 0 0 0 0))
+  )
+  (wire (pts (xy 164.465 42.545) (xy 168.275 42.545))
+    (stroke (width 0) (type default) (color 0 0 0 0))
+  )
+  (wire (pts (xy 180.34 58.42) (xy 180.34 59.69))
+    (stroke (width 0) (type default) (color 0 0 0 0))
+  )
+  (wire (pts (xy 71.755 48.895) (xy 71.755 60.325))
+    (stroke (width 0) (type default) (color 0 0 0 0))
+  )
+  (wire (pts (xy 96.52 76.454) (xy 96.52 85.09))
+    (stroke (width 0) (type default) (color 0 0 0 0))
+  )
+  (wire (pts (xy 199.39 78.74) (xy 199.39 52.705))
+    (stroke (width 0) (type default) (color 0 0 0 0))
+  )
+  (wire (pts (xy 233.045 68.58) (xy 233.045 67.945))
+    (stroke (width 0) (type default) (color 0 0 0 0))
+  )
+  (wire (pts (xy 158.877 58.039) (xy 156.21 58.039))
+    (stroke (width 0) (type default) (color 0 0 0 0))
+  )
   (wire (pts (xy 49.022 92.329) (xy 49.022 97.409))
-    (stroke (width 0) (type default) (color 0 0 0 0))
-  )
-  (wire (pts (xy 202.057 46.482) (xy 187.325 46.482))
-    (stroke (width 0) (type default) (color 0 0 0 0))
-  )
-  (wire (pts (xy 117.348 54.102) (xy 122.555 54.102))
-    (stroke (width 0) (type default) (color 0 0 0 0))
-  )
-  (wire (pts (xy 148.59 52.197) (xy 148.59 61.595))
-    (stroke (width 0) (type default) (color 0 0 0 0))
-  )
-  (wire (pts (xy 156.21 42.545) (xy 156.21 58.039))
-    (stroke (width 0) (type default) (color 0 0 0 0))
-  )
-  (wire (pts (xy 122.555 54.102) (xy 122.555 61.595))
-    (stroke (width 0) (type default) (color 0 0 0 0))
-  )
-  (wire (pts (xy 196.85 51.054) (xy 196.85 76.2))
-    (stroke (width 0) (type default) (color 0 0 0 0))
-  )
-  (wire (pts (xy 164.465 42.545) (xy 168.275 42.545))
-    (stroke (width 0) (type default) (color 0 0 0 0))
-  )
-  (wire (pts (xy 180.34 58.42) (xy 180.34 59.69))
-    (stroke (width 0) (type default) (color 0 0 0 0))
-  )
-  (wire (pts (xy 71.755 48.895) (xy 71.755 60.325))
-    (stroke (width 0) (type default) (color 0 0 0 0))
-  )
-  (wire (pts (xy 96.52 76.454) (xy 96.52 85.09))
-    (stroke (width 0) (type default) (color 0 0 0 0))
-  )
-  (wire (pts (xy 199.39 78.74) (xy 199.39 52.705))
-    (stroke (width 0) (type default) (color 0 0 0 0))
-  )
-  (wire (pts (xy 233.045 68.58) (xy 233.045 67.945))
-    (stroke (width 0) (type default) (color 0 0 0 0))
-  )
-  (wire (pts (xy 158.877 58.039) (xy 156.21 58.039))
     (stroke (width 0) (type default) (color 0 0 0 0))
   )
@@
     (pin "2")
   )
-  (symbol (lib_id "centrifuge_symbols:+3V3_MCU") (at 49.022 79.629 0) (unit 1)
-    (in_bom yes) (on_board yes) (fields_autoplaced)
-    (property "Reference" "#PWR0238" (id 0) (at 49.022 83.439 0)
-      (effects (font (size 1.27 1.27)) hide)
-    )
-    (property "Value" "+3V3_MCU" (id 1) (at 49.022 73.914 0))
-    (property "Footprint" "" (id 2) (at 49.022 79.629 0)
-      (effects (font (size 1.27 1.27)) hide)
-    )
-    (property "Datasheet" "" (id 3) (at 49.022 79.629 0)
+  (symbol (lib_id "centrifuge_symbols:+3V3_MCU") (at 41.402 79.629 0) (unit 1)
+    (in_bom yes) (on_board yes) (fields_autoplaced)
+    (property "Reference" "#PWR0238" (id 0) (at 41.402 83.439 0)
+      (effects (font (size 1.27 1.27)) hide)
+    )
+    (property "Value" "+3V3_MCU" (id 1) (at 41.402 73.914 0))
+    (property "Footprint" "" (id 2) (at 41.402 79.629 0)
+      (effects (font (size 1.27 1.27)) hide)
+    )
+    (property "Datasheet" "" (id 3) (at 41.402 79.629 0)
       (effects (font (size 1.27 1.27)) hide)
     )
@@
     (pin "1")
   )
-  (symbol (lib_id "centrifuge_symbols:+3V3A_FPGA") (at 64.135 48.895 0) (unit 1)
+  (symbol (lib_id "centrifuge_symbols:+1V8_FPGA") (at 64.135 48.895 0) (unit 1)
     (in_bom yes) (on_board yes) (fields_autoplaced)
     (property "Reference" "#PWR0501" (id 0) (at 67.945 50.165 0)
       (effects (font (size 1.27 1.27)) hide)
     )
-    (property "Value" "+3V3A_FPGA" (id 1) (at 64.135 45.339 90)
+    (property "Value" "+1V8_FPGA" (id 1) (at 64.135 45.339 90)
       (effects (font (size 1.27 1.27)) (justify left))
     )
@@
     (pin "1")
   )
-  (symbol (lib_id "centrifuge_symbols:+3V3_FPGA") (at 74.295 48.895 0) (unit 1)
+  (symbol (lib_id "centrifuge_symbols:+5V_FPGA") (at 74.295 48.895 0) (unit 1)
     (in_bom yes) (on_board yes) (fields_autoplaced)
     (property "Reference" "#PWR0508" (id 0) (at 74.295 52.705 0)
       (effects (font (size 1.27 1.27)) hide)
     )
-    (property "Value" "+3V3_FPGA" (id 1) (at 74.295 45.339 90)
+    (property "Value" "+5V_FPGA" (id 1) (at 74.295 45.339 90)
       (effects (font (size 1.27 1.27)) (justify left))
     )
@@
     (pin "2")
   )
-  (symbol (lib_id "centrifuge_symbols:+5V_FPGA") (at 76.835 48.895 0) (unit 1)
+  (symbol (lib_id "centrifuge_symbols:+3V3A_FPGA") (at 76.835 48.895 0) (unit 1)
     (in_bom yes) (on_board yes) (fields_autoplaced)
     (property "Reference" "#PWR0510" (id 0) (at 76.835 52.705 0)
       (effects (font (size 1.27 1.27)) hide)
     )
-    (property "Value" "+5V_FPGA" (id 1) (at 76.835 45.339 90)
+    (property "Value" "+3V3A_FPGA" (id 1) (at 76.835 45.339 90)
       (effects (font (size 1.27 1.27)) (justify left))
     )
@@
     (pin "1")
   )
-  (symbol (lib_id "centrifuge_symbols:+1V8_FPGA") (at 71.755 48.895 0) (unit 1)
+  (symbol (lib_id "centrifuge_symbols:+1V9_FPGA") (at 71.755 48.895 0) (unit 1)
     (in_bom yes) (on_board yes) (fields_autoplaced)
     (property "Reference" "#PWR0506" (id 0) (at 71.755 52.705 0)
       (effects (font (size 1.27 1.27)) hide)
     )
-    (property "Value" "+1V8_FPGA" (id 1) (at 71.755 45.339 90)
+    (property "Value" "+1V9_FPGA" (id 1) (at 71.755 43.18 90)
       (effects (font (size 1.27 1.27)) (justify left))
     )
@@
     (pin "2")
   )
-  (symbol (lib_id "centrifuge_symbols:+1V9_FPGA") (at 66.675 48.895 0) (unit 1)
+  (symbol (lib_id "centrifuge_symbols:+3V3_FPGA") (at 66.675 48.895 0) (unit 1)
     (in_bom yes) (on_board yes) (fields_autoplaced)
     (property "Reference" "#PWR0502" (id 0) (at 66.675 52.705 0)
       (effects (font (size 1.27 1.27)) hide)
     )
-    (property "Value" "+1V9_FPGA" (id 1) (at 66.675 43.18 90)
+    (property "Value" "+3V3_FPGA" (id 1) (at 66.675 45.339 90)
       (effects (font (size 1.27 1.27)) (justify left))
     )
@@
       (effects (font (size 1.27 1.27)) (justify left top))
     )
-    (pin "3V3ADC" output (at 64.135 113.03 90)
+    (pin "3V3ADC" output (at 76.835 113.03 90)
       (effects (font (size 1.27 1.27)) (justify right))
     )
-    (pin "3V3" output (at 74.295 113.03 90)
+    (pin "3V3" output (at 66.675 113.03 90)
       (effects (font (size 1.27 1.27)) (justify right))
     )
@@
       (effects (font (size 1.27 1.27)) (justify right))
     )
-    (pin "1V8" output (at 71.755 113.03 90)
+    (pin "1V8" output (at 64.135 113.03 90)
       (effects (font (size 1.27 1.27)) (justify right))
     )
-    (pin "1V9" output (at 66.675 113.03 90)
+    (pin "1V9" output (at 71.755 113.03 90)
       (effects (font (size 1.27 1.27)) (justify right))
     )
-    (pin "5V0" output (at 76.835 113.03 90)
+    (pin "5V0" output (at 74.295 113.03 90)
       (effects (font (size 1.27 1.27)) (justify right))
     )
