File: centrifuge_combined/mcu_part/centrifuge_mcu.kicad_sch (KiCad schematic)
At the start: 16 parts, among them J501 Conn_02x06_Odd_Even, J503 MCU_extra, J505 FPGA_SPI, J506 DDCI2C2, J507 ADC_I2C, J508 ADC_RST, J516 Conn_02x06_Odd_Even, J517 DDCI2C1, U501 DFR0555, U502 LCD16x2L

Commit message: change resistor values to have to 2k2, and also make I2C hopefully work
Parts:
- R501, R502, R503, R504: value 2.2k -> 10k
- R505, R506: value 2.2k -> 4.7k
Connections:
- net I2C0_SCL#1 renamed SCL_MCU_SL2
- net I2C0_SCL#2 renamed SCL_MCU_SL1
- net I2C0_SDA#1 renamed SDA_MCU_SL2
- net I2C0_SDA#2 renamed SDA_MCU_SL1
Other:
- note added: "Used to be 2.2k"
Changed lines of the file:
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@@
     (stroke (width 0) (type default) (color 0 0 0 0))
+  )
+  (text "Used to be 2.2k" (at 170.688 68.072 0)
+    (effects (font (size 1.27 1.27)) (justify left bottom))
+  )
+  (text "Used to be 2.2k" (at 166.37 47.752 90)
+    (effects (font (size 1.27 1.27)) (justify left bottom))
   )
   (text "LCD screen" (at 238.125 57.15 0)
@@
     (effects (font (size 1.27 1.27)) (justify left))
   )
-  (hierarchical_label "I2C0_SCL#2" (shape bidirectional) (at 158.877 52.197 0)
+  (hierarchical_label "SCL_MCU_SL1" (shape bidirectional) (at 158.877 52.197 0)
     (effects (font (size 1.27 1.27)) (justify left))
   )
@@
     (effects (font (size 1.27 1.27)) (justify right))
   )
-  (hierarchical_label "I2C0_SDA#2" (shape bidirectional) (at 158.877 54.229 0)
+  (hierarchical_label "SDA_MCU_SL1" (shape bidirectional) (at 158.877 54.229 0)
     (effects (font (size 1.27 1.27)) (justify left))
   )
@@
     (effects (font (size 1.27 1.27)) (justify left))
   )
-  (hierarchical_label "I2C0_SDA#1" (shape bidirectional) (at 158.877 58.039 0)
-    (effects (font (size 1.27 1.27)) (justify left))
-  )
-  (hierarchical_label "I2C0_SCL#1" (shape bidirectional) (at 158.877 56.388 0)
+  (hierarchical_label "SDA_MCU_SL2" (shape bidirectional) (at 158.877 58.039 0)
+    (effects (font (size 1.27 1.27)) (justify left))
+  )
+  (hierarchical_label "SCL_MCU_SL2" (shape bidirectional) (at 158.877 56.388 0)
     (effects (font (size 1.27 1.27)) (justify left))
   )
@@
     (in_bom yes) (on_board yes)
     (property "Reference" "R503" (id 0) (at 160.655 40.64 90))
-    (property "Value" "2.2k" (id 1) (at 160.655 42.545 90))
+    (property "Value" "10k" (id 1) (at 160.655 42.545 90))
     (property "Footprint" "Resistor_SMD:R_0805_2012Metric_Pad1.20x1.40mm_HandSolder" (id 2) (at 160.655 44.323 90)
       (effects (font (size 1.27 1.27)) hide)
@@
     (in_bom yes) (on_board yes)
     (property "Reference" "R505" (id 0) (at 176.53 63.5 90))
-    (property "Value" "2.2k" (id 1) (at 174.625 63.5 90))
+    (property "Value" "4.7k" (id 1) (at 174.625 63.5 90))
     (property "Footprint" "Resistor_SMD:R_0805_2012Metric_Pad1.20x1.40mm_HandSolder" (id 2) (at 172.847 63.5 90)
       (effects (font (size 1.27 1.27)) hide)
@@
     (in_bom yes) (on_board yes)
     (property "Reference" "R506" (id 0) (at 182.245 63.5 90))
-    (property "Value" "2.2k" (id 1) (at 180.34 63.5 90))
+    (property "Value" "4.7k" (id 1) (at 180.34 63.5 90))
     (property "Footprint" "Resistor_SMD:R_0805_2012Metric_Pad1.20x1.40mm_HandSolder" (id 2) (at 178.562 63.5 90)
       (effects (font (size 1.27 1.27)) hide)
@@
     (in_bom yes) (on_board yes)
     (property "Reference" "R504" (id 0) (at 160.655 45.085 90))
-    (property "Value" "2.2k" (id 1) (at 160.655 46.99 90))
+    (property "Value" "10k" (id 1) (at 160.655 46.99 90))
     (property "Footprint" "Resistor_SMD:R_0805_2012Metric_Pad1.20x1.40mm_HandSolder" (id 2) (at 160.655 48.768 90)
       (effects (font (size 1.27 1.27)) hide)
@@
     (in_bom yes) (on_board yes)
     (property "Reference" "R501" (id 0) (at 160.655 31.115 90))
-    (property "Value" "2.2k" (id 1) (at 160.655 33.02 90))
+    (property "Value" "10k" (id 1) (at 160.655 33.02 90))
     (property "Footprint" "Resistor_SMD:R_0805_2012Metric_Pad1.20x1.40mm_HandSolder" (id 2) (at 160.655 34.798 90)
       (effects (font (size 1.27 1.27)) hide)
@@
     (in_bom yes) (on_board yes)
     (property "Reference" "R502" (id 0) (at 160.655 35.56 90))
-    (property "Value" "2.2k" (id 1) (at 160.655 37.465 90))
+    (property "Value" "10k" (id 1) (at 160.655 37.465 90))
     (property "Footprint" "Resistor_SMD:R_0805_2012Metric_Pad1.20x1.40mm_HandSolder" (id 2) (at 160.655 39.243 90)
       (effects (font (size 1.27 1.27)) hide)

Commit message: change the names of some named wires in the schematic, to make numbering more consistent
Connections:
- net ADC0_RST renamed ADC2_RST
Other:
- sheet MCU ports: added ADC2_RST; removed ADC0_RST
Changed lines of the file:
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@@
     (effects (font (size 1.27 1.27)) (justify left))
   )
-  (hierarchical_label "ADC0_RST" (shape output) (at 202.057 51.054 0)
+  (hierarchical_label "ADC2_RST" (shape output) (at 202.057 51.054 0)
     (effects (font (size 1.27 1.27)) (justify left))
   )
@@
       (effects (font (size 1.27 1.27)) (justify right))
     )
-    (pin "ADC0_RST" bidirectional (at 168.91 76.2 0)
-      (effects (font (size 1.27 1.27)) (justify right))
-    )
+    (pin "ADC2_RST" bidirectional (at 168.91 76.2 0)
+      (effects (font (size 1.27 1.27)) (justify right))
+    )
