File: centrifuge_combined/mcu_part/mcu.kicad_sch (KiCad schematic)
At the start: 22 parts, among them J514 DEBUG, J515 Extra MCU GPIO, Q502 Q_NMOS_GSD, U506 EFM32GG990F1024, Y501 VXM7-1366-48M0000000

Commit message: Fixed Elprint complaints and JTAG VREF problems+config flash CS
Parts:
- C539, C550: Order Page https://no.mouser.com/ProductDetail/Samsung-Electro-Mechani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 -> (none); Purchase (none) -> https://www.digikey.no/no/products/detail/yageo/CC0805MKX5R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
- C540: Order Page https://no.mouser.com/ProductDetail/Walsin/0805X105K100CT?q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 -> (none); Purchase (none) -> https://www.digikey.no/no/products/detail/kemet/C0805C105J4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
Other:
- note added: "Extra MCU-FPGA IO"
- note removed: "Extra MCU GPIO"
Changed lines of the file:
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@@
   (title_block
     (title "VGA Centrifuge")
-    (date "2022-10-03")
-    (rev "R3")
+    (date "2022-10-05")
+    (rev "R4")
     (comment 1 "Author: Håvard Krogstie")
     (comment 2 "MCU interfaces")
@@
     (effects (font (size 1.27 1.27)) (justify left bottom))
   )
-  (text "Extra MCU GPIO" (at 174.625 43.815 0)
+  (text "Extra MCU-FPGA IO" (at 174.625 43.815 0)
     (effects (font (size 1.27 1.27)) (justify left bottom))
   )
@@
       (effects (font (size 1.27 1.27)) hide)
     )
-    (property "Purchase" "" (id 4) (at 163.195 180.34 0)
-      (effects (font (size 1.27 1.27)) hide)
-    )
-    (property "Order Page" "https://no.mouser.com/ProductDetail/Samsung-Electro-Mechanics/CL21A106KOQNNNE?qs=sGAEpiMZZMsh%252B1woXyUXj7iNKXiFkBmwjufexzBEAvI%3D" (id 5) (at 163.195 180.34 0)
+    (property "Purchase" "https://www.digikey.no/no/products/detail/yageo/CC0805MKX5R7BB106/5884266" (id 4) (at 163.195 180.34 0)
       (effects (font (size 1.27 1.27)) hide)
     )
@@
       (effects (font (size 1.27 1.27)) hide)
     )
-    (property "Purchase" "" (id 4) (at 74.93 179.705 0)
-      (effects (font (size 1.27 1.27)) hide)
-    )
-    (property "Order Page" "https://no.mouser.com/ProductDetail/Samsung-Electro-Mechanics/CL21A106KOQNNNE?qs=sGAEpiMZZMsh%252B1woXyUXj7iNKXiFkBmwjufexzBEAvI%3D" (id 5) (at 74.93 179.705 0)
+    (property "Purchase" "https://www.digikey.no/no/products/detail/yageo/CC0805MKX5R7BB106/5884266" (id 4) (at 74.93 179.705 0)
       (effects (font (size 1.27 1.27)) hide)
     )
@@
       (effects (font (size 1.27 1.27)) hide)
     )
-    (property "Purchase" "" (id 4) (at 94.615 37.465 0)
-      (effects (font (size 1.27 1.27)) hide)
-    )
-    (property "Order Page" "https://no.mouser.com/ProductDetail/Walsin/0805X105K100CT?qs=sGAEpiMZZMsh%252B1woXyUXj6GIMbU2VNPkBXHihtGsekQ%3D" (id 5) (at 94.615 37.465 0)
-      (effects (font (size 1.27 1.27)) hide)
-    )
+    (property "Purchase" "https://www.digikey.no/no/products/detail/kemet/C0805C105J4REC7800/8643700" (id 4) (at 94.615 37.465 0)
+      (effects (font (size 1.27 1.27)) hide)
+    )
