File: centrifuge_combined/mcu_part/mcu.kicad_sch (KiCad schematic)
At the start: 22 parts, among them J514 DEBUG, J515 Extra MCU GPIO, Q502 Q_NMOS_GSD, U506 EFM32GG990F1024, Y501 VXM7-1366-48M0000000

Commit message: Fixed missing footprints, added decoupling capacitors, adjusted board edges
Parts:
- C536, C537, C538, C539, C540, C541, C542, C543, C544, C545, C546, C547, C548, C549, C550: footprint (none) -> Capacitor_SMD:C_0805_2012Metric_Pad1.18x1.45mm_HandSolder
- D501: footprint (none) -> Diode_SMD:D_0805_2012Metric_Pad1.15x1.40mm_HandSolder
- J514: footprint (none) -> Connector_PinHeader_1.27mm:PinHeader_2x10_P1.27mm_Vertical
- J515: footprint (none) -> Connector_PinHeader_2.54mm:PinHeader_2x04_P2.54mm_Vertical
- Q502: footprint (none) -> Package_TO_SOT_SMD:SOT-323_SC-70_Handsoldering
- R528: footprint (none) -> Resistor_SMD:R_0805_2012Metric_Pad1.20x1.40mm_HandSolder
- U506: footprint (none) -> centrifuge_mcu:BGA-112_9.0x9.0mm_Layout11x11_P0.8mm_Ball0.4mm_Pad0.35mm_NSMD
- Y501: footprint (none) -> centrifuge_mcu:Crystal_SMD_TXC_7M-4Pin_3.2x2.5mm_TIGHT
Changed lines of the file:
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@@
     (title "VGA Centrifuge")
     (date "2022-10-03")
-    (rev "R2")
+    (rev "R3")
+    (comment 1 "Author: Håvard Krogstie")
+    (comment 2 "MCU interfaces")
   )
   (junction (at 144.145 176.53) (diameter 0) (color 0 0 0 0)
@@
       (effects (font (size 1.27 1.27)) (justify left))
     )
-    (property "Footprint" "" (id 2) (at 121.92 93.345 0)
+    (property "Footprint" "centrifuge_mcu:BGA-112_9.0x9.0mm_Layout11x11_P0.8mm_Ball0.4mm_Pad0.35mm_NSMD" (id 2) (at 121.92 93.345 0)
       (effects (font (size 1.27 1.27)) hide)
     )
@@
       (effects (font (size 1.27 1.27)) (justify left))
     )
-    (property "Footprint" "" (id 2) (at 154.6352 184.15 0)
+    (property "Footprint" "Capacitor_SMD:C_0805_2012Metric_Pad1.18x1.45mm_HandSolder" (id 2) (at 154.6352 184.15 0)
       (effects (font (size 1.27 1.27)) hide)
     )
@@
     (property "Reference" "Y501" (id 0) (at 118.745 46.355 0))
     (property "Value" "VXM7-1366-48M0000000" (id 1) (at 119.38 48.895 0))
-    (property "Footprint" "" (id 2) (at 119.38 59.055 0)
+    (property "Footprint" "centrifuge_mcu:Crystal_SMD_TXC_7M-4Pin_3.2x2.5mm_TIGHT" (id 2) (at 119.38 59.055 0)
       (effects (font (size 1.27 1.27)) hide)
     )
@@
       (effects (font (size 1.27 1.27)) (justify left))
     )
-    (property "Footprint" "" (id 2) (at 164.1602 184.15 0)
+    (property "Footprint" "Capacitor_SMD:C_0805_2012Metric_Pad1.18x1.45mm_HandSolder" (id 2) (at 164.1602 184.15 0)
       (effects (font (size 1.27 1.27)) hide)
     )
@@
       (effects (font (size 1.27 1.27)) (justify left))
     )
-    (property "Footprint" "" (id 2) (at 116.5352 184.15 0)
+    (property "Footprint" "Capacitor_SMD:C_0805_2012Metric_Pad1.18x1.45mm_HandSolder" (id 2) (at 116.5352 184.15 0)
       (effects (font (size 1.27 1.27)) hide)
     )
@@
       (effects (font (size 1.27 1.27)) hide)
     )
-    (property "Footprint" "" (id 2) (at 29.845 145.415 0)
+    (property "Footprint" "Connector_PinHeader_1.27mm:PinHeader_2x10_P1.27mm_Vertical" (id 2) (at 29.845 145.415 0)
       (effects (font (size 1.27 1.27)) hide)
     )
@@
       (effects (font (size 1.27 1.27)) (justify left))
     )
-    (property "Footprint" "" (id 2) (at 97.4852 184.15 0)
+    (property "Footprint" "Capacitor_SMD:C_0805_2012Metric_Pad1.18x1.45mm_HandSolder" (id 2) (at 97.4852 184.15 0)
       (effects (font (size 1.27 1.27)) hide)
     )
@@
       (effects (font (size 1.27 1.27)) (justify left))
     )
-    (property "Footprint" "" (id 2) (at 66.3702 183.515 0)
+    (property "Footprint" "Capacitor_SMD:C_0805_2012Metric_Pad1.18x1.45mm_HandSolder" (id 2) (at 66.3702 183.515 0)
       (effects (font (size 1.27 1.27)) hide)
     )
@@
       (effects (font (size 1.27 1.27)) (justify left))
     )
-    (property "Footprint" "" (id 2) (at 126.0602 184.15 0)
+    (property "Footprint" "Capacitor_SMD:C_0805_2012Metric_Pad1.18x1.45mm_HandSolder" (id 2) (at 126.0602 184.15 0)
       (effects (font (size 1.27 1.27)) hide)
     )
@@
       (effects (font (size 1.27 1.27)) (justify left))
     )
-    (property "Footprint" "" (id 2) (at 147.32 5.08 0)
+    (property "Footprint" "centrifuge_mcu:BGA-112_9.0x9.0mm_Layout11x11_P0.8mm_Ball0.4mm_Pad0.35mm_NSMD" (id 2) (at 147.32 5.08 0)
       (effects (font (size 1.27 1.27)) hide)
     )
@@
       (effects (font (size 1.27 1.27)) (justify left))
     )
-    (property "Footprint" "" (id 2) (at 56.8452 183.515 0)
+    (property "Footprint" "Capacitor_SMD:C_0805_2012Metric_Pad1.18x1.45mm_HandSolder" (id 2) (at 56.8452 183.515 0)
       (effects (font (size 1.27 1.27)) hide)
     )
@@
     (property "Reference" "J515" (id 0) (at 172.72 107.95 0))
     (property "Value" "Extra MCU GPIO" (id 1) (at 175.26 125.73 0))
-    (property "Footprint" "" (id 2) (at 171.45 115.57 0)
+    (property "Footprint" "Connector_PinHeader_2.54mm:PinHeader_2x04_P2.54mm_Vertical" (id 2) (at 171.45 115.57 0)
       (effects (font (size 1.27 1.27)) hide)
     )
@@
       (effects (font (size 1.27 1.27)) (justify left))
     )
-    (property "Footprint" "" (id 2) (at 107.0102 184.15 0)
+    (property "Footprint" "Capacitor_SMD:C_0805_2012Metric_Pad1.18x1.45mm_HandSolder" (id 2) (at 107.0102 184.15 0)
       (effects (font (size 1.27 1.27)) hide)
     )
@@
       (effects (font (size 1.27 1.27)) (justify left))
     )
-    (property "Footprint" "" (id 2) (at 75.8952 183.515 0)
+    (property "Footprint" "Capacitor_SMD:C_0805_2012Metric_Pad1.18x1.45mm_HandSolder" (id 2) (at 75.8952 183.515 0)
       (effects (font (size 1.27 1.27)) hide)
     )
@@
       (effects (font (size 1.27 1.27)) (justify left))
     )
-    (property "Footprint" "" (id 2) (at 135.5852 184.15 0)
+    (property "Footprint" "Capacitor_SMD:C_0805_2012Metric_Pad1.18x1.45mm_HandSolder" (id 2) (at 135.5852 184.15 0)
       (effects (font (size 1.27 1.27)) hide)
     )
@@
     (property "Reference" "U506" (id 0) (at 62.865 24.13 0))
     (property "Value" "EFM32GG990F1024" (id 1) (at 62.865 26.67 0))
-    (property "Footprint" "" (id 2) (at 63.5 15.24 0)
+    (property "Footprint" "centrifuge_mcu:BGA-112_9.0x9.0mm_Layout11x11_P0.8mm_Ball0.4mm_Pad0.35mm_NSMD" (id 2) (at 63.5 15.24 0)
       (effects (font (size 1.27 1.27)) hide)
     )
@@
     (property "Reference" "U506" (id 0) (at 215.265 39.37 0))
     (property "Value" "EFM32GG990F1024" (id 1) (at 215.265 41.91 0))
-    (property "Footprint" "" (id 2) (at 213.995 46.355 0)
+    (property "Footprint" "centrifuge_mcu:BGA-112_9.0x9.0mm_Layout11x11_P0.8mm_Ball0.4mm_Pad0.35mm_NSMD" (id 2) (at 213.995 46.355 0)
       (effects (font (size 1.27 1.27)) hide)
     )
@@
       (effects (font (size 1.27 1.27)) (justify left))
     )
-    (property "Footprint" "" (id 2) (at 126.0602 69.85 0)
+    (property "Footprint" "Capacitor_SMD:C_0805_2012Metric_Pad1.18x1.45mm_HandSolder" (id 2) (at 126.0602 69.85 0)
       (effects (font (size 1.27 1.27)) hide)
     )
@@
       (effects (font (size 1.27 1.27)) (justify left))
     )
-    (property "Footprint" "" (id 2) (at 145.1102 184.15 0)
+    (property "Footprint" "Capacitor_SMD:C_0805_2012Metric_Pad1.18x1.45mm_HandSolder" (id 2) (at 145.1102 184.15 0)
       (effects (font (size 1.27 1.27)) hide)
     )
@@
       (effects (font (size 1.27 1.27)) (justify left))
     )
-    (property "Footprint" "" (id 2) (at 47.3202 183.515 0)
+    (property "Footprint" "Capacitor_SMD:C_0805_2012Metric_Pad1.18x1.45mm_HandSolder" (id 2) (at 47.3202 183.515 0)
       (effects (font (size 1.27 1.27)) hide)
     )
@@
       (effects (font (size 1.27 1.27)) (justify right))
     )
-    (property "Footprint" "" (id 2) (at 146.05 87.63 0)
+    (property "Footprint" "Diode_SMD:D_0805_2012Metric_Pad1.15x1.40mm_HandSolder" (id 2) (at 146.05 87.63 0)
       (effects (font (size 1.27 1.27)) hide)
     )
@@
       (effects (font (size 1.27 1.27)) (justify left))
     )
-    (property "Footprint" "" (id 2) (at 113.3602 69.85 0)
+    (property "Footprint" "Capacitor_SMD:C_0805_2012Metric_Pad1.18x1.45mm_HandSolder" (id 2) (at 113.3602 69.85 0)
       (effects (font (size 1.27 1.27)) hide)
     )
@@
       (effects (font (size 1.27 1.27)) (justify left))
     )
-    (property "Footprint" "" (id 2) (at 144.272 78.74 90)
+    (property "Footprint" "Resistor_SMD:R_0805_2012Metric_Pad1.20x1.40mm_HandSolder" (id 2) (at 144.272 78.74 90)
       (effects (font (size 1.27 1.27)) hide)
     )
@@
       (effects (font (size 1.27 1.27)) (justify right))
     )
-    (property "Footprint" "" (id 2) (at 93.6498 33.655 0)
+    (property "Footprint" "Capacitor_SMD:C_0805_2012Metric_Pad1.18x1.45mm_HandSolder" (id 2) (at 93.6498 33.655 0)
       (effects (font (size 1.27 1.27)) hide)
     )
@@
       (effects (font (size 1.27 1.27)) (justify left))
     )
-    (property "Footprint" "" (id 2) (at 143.51 97.155 0)
-      (effects (font (size 1.27 1.27)) hide)
-    )
+    (property "Footprint" "Package_TO_SOT_SMD:SOT-323_SC-70_Handsoldering" (id 2) (at 143.51 97.155 0)
+      (effects (font (size 1.27 1.27)) hide)
+    )

Commit message: remove digikey links to products that we already buy from mouser, add mouser link instead
Parts:
- C539, C550: Order Page (none) -> https://no.mouser.com/ProductDetail/Samsung-Electro-Mechani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; Purchase https://www.digikey.no/no/products/detail/yageo/CC0805MKX5R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 -> (none)
- C540: Order Page (none) -> https://no.mouser.com/ProductDetail/Walsin/0805X105K100CT?q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; Purchase https://www.digikey.no/no/products/detail/kemet/C0805C105J4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 -> (none)
Changed lines of the file:
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@@
       (effects (font (size 1.27 1.27)) hide)
     )
-    (property "Purchase" "https://www.digikey.no/no/products/detail/yageo/CC0805MKX5R7BB106/5884266" (id 4) (at 163.195 180.34 0)
+    (property "Purchase" "" (id 4) (at 163.195 180.34 0)
+      (effects (font (size 1.27 1.27)) hide)
+    )
+    (property "Order Page" "https://no.mouser.com/ProductDetail/Samsung-Electro-Mechanics/CL21A106KOQNNNE?qs=sGAEpiMZZMsh%252B1woXyUXj7iNKXiFkBmwjufexzBEAvI%3D" (id 5) (at 163.195 180.34 0)
       (effects (font (size 1.27 1.27)) hide)
     )
@@
       (effects (font (size 1.27 1.27)) hide)
     )
-    (property "Purchase" "https://www.digikey.no/no/products/detail/yageo/CC0805MKX5R7BB106/5884266" (id 4) (at 74.93 179.705 0)
+    (property "Purchase" "" (id 4) (at 74.93 179.705 0)
+      (effects (font (size 1.27 1.27)) hide)
+    )
+    (property "Order Page" "https://no.mouser.com/ProductDetail/Samsung-Electro-Mechanics/CL21A106KOQNNNE?qs=sGAEpiMZZMsh%252B1woXyUXj7iNKXiFkBmwjufexzBEAvI%3D" (id 5) (at 74.93 179.705 0)
       (effects (font (size 1.27 1.27)) hide)
     )
@@
       (effects (font (size 1.27 1.27)) hide)
     )
-    (property "Purchase" "https://www.digikey.no/no/products/detail/kemet/C0805C105J4REC7800/8643700" (id 4) (at 94.615 37.465 0)
-      (effects (font (size 1.27 1.27)) hide)
-    )
+    (property "Purchase" "" (id 4) (at 94.615 37.465 0)
+      (effects (font (size 1.27 1.27)) hide)
+    )
+    (property "Order Page" "https://no.mouser.com/ProductDetail/Walsin/0805X105K100CT?qs=sGAEpiMZZMsh%252B1woXyUXj6GIMbU2VNPkBXHihtGsekQ%3D" (id 5) (at 94.615 37.465 0)
+      (effects (font (size 1.27 1.27)) hide)
+    )

Commit message: fix elprint complaints, except intranet clearance, also widen some traces
Other:
- note added: "Extra MCU GPIO"
- note removed: "Extra MCU-FPGA IO"
Changed lines of the file:
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@@
     (effects (font (size 1.27 1.27)) (justify left bottom))
   )
-  (text "Extra MCU-FPGA IO" (at 174.625 43.815 0)
+  (text "Extra MCU GPIO" (at 174.625 43.815 0)
     (effects (font (size 1.27 1.27)) (justify left bottom))
   )

Commit message: change the names of some named wires in the schematic, to make numbering more consistent
Connections:
- net ADC0_RST renamed ADC2_RST
Other:
- note added: "ADC1's DDC I2C"
- note added: "ADC2's DDC I2C"
- note removed: "DDC I2C x2"
Changed lines of the file:
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@@
     (effects (font (size 1.27 1.27)) (justify left bottom))
   )
-  (text "DDC I2C x2" (at 240.03 105.41 0)
+  (text "ADC2's DDC I2C" (at 240.03 105.41 0)
     (effects (font (size 1.27 1.27)) (justify left bottom))
   )
@@
   )
   (text "Power" (at 59.69 22.225 0)
+    (effects (font (size 1.27 1.27)) (justify left bottom))
+  )
+  (text "ADC1's DDC I2C" (at 239.522 116.078 0)
     (effects (font (size 1.27 1.27)) (justify left bottom))
   )
@@
     (effects (font (size 1.27 1.27)) (justify left))
   )
-  (hierarchical_label "ADC0_RST" (shape bidirectional) (at 248.92 140.335 0)
+  (hierarchical_label "ADC2_RST" (shape bidirectional) (at 248.92 140.335 0)
     (effects (font (size 1.27 1.27)) (justify left))
   )
