File: centrifuge_combined/mcu_part/power_circuit.kicad_sch (KiCad schematic)
At the start: 66 parts, among them J509 USB_B_Micro, J510 Barrel_Jack, J511 PowerIn, J512 PowerPads, Q501 Q_PMOS_DGS, U503 TPS54294, U504 TPS54294, U505 TPS54294

Commit message: Fixed Elprint complaints and JTAG VREF problems+config flash CS
Parts:
- C517, C518, C519: Order Page https://no.mouser.com/ProductDetail/Walsin/0805X105K100CT?q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 -> (none); Purchase (none) -> https://www.digikey.no/no/products/detail/kemet/C0805C105J4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
- R514, R515, R516: Order Page https://no.mouser.com/ProductDetail/YAGEO/RC0805FR-1310KL?q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 -> (none); Purchase (none) -> https://www.digikey.no/no/products/detail/yageo/AC0805FR-07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
Changed lines of the file:
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@@
   (title_block
     (title "VGA Centrifuge")
-    (date "2022-10-03")
-    (rev "R3")
+    (date "2022-10-05")
+    (rev "R4")
     (comment 1 "Author: Håvard Krogstie")
     (comment 2 "Power Supply")
@@
       (effects (font (size 1.27 1.27)) hide)
     )
-    (property "Purchase" "" (id 4) (at 203.2 43.815 0)
-      (effects (font (size 1.27 1.27)) hide)
-    )
-    (property "Order Page" "https://no.mouser.com/ProductDetail/YAGEO/RC0805FR-1310KL?qs=sGAEpiMZZMtlubZbdhIBIHucEnbnlIRRGobQQ23C9vc%3D" (id 5) (at 203.2 43.815 0)
+    (property "Purchase" "https://www.digikey.no/no/products/detail/yageo/AC0805FR-07100KL/5896520" (id 4) (at 203.2 43.815 0)
       (effects (font (size 1.27 1.27)) hide)
     )
@@
       (effects (font (size 1.27 1.27)) hide)
     )
-    (property "Purchase" "" (id 4) (at 197.485 100.33 0)
-      (effects (font (size 1.27 1.27)) hide)
-    )
-    (property "Order Page" "https://no.mouser.com/ProductDetail/Walsin/0805X105K100CT?qs=sGAEpiMZZMsh%252B1woXyUXj6GIMbU2VNPkBXHihtGsekQ%3D" (id 5) (at 197.485 100.33 0)
+    (property "Purchase" "https://www.digikey.no/no/products/detail/kemet/C0805C105J4REC7800/8643700" (id 4) (at 197.485 100.33 0)
       (effects (font (size 1.27 1.27)) hide)
     )
@@
       (effects (font (size 1.27 1.27)) hide)
     )
-    (property "Purchase" "" (id 4) (at 198.12 153.67 0)
-      (effects (font (size 1.27 1.27)) hide)
-    )
-    (property "Order Page" "https://no.mouser.com/ProductDetail/Walsin/0805X105K100CT?qs=sGAEpiMZZMsh%252B1woXyUXj6GIMbU2VNPkBXHihtGsekQ%3D" (id 5) (at 198.12 153.67 0)
+    (property "Purchase" "https://www.digikey.no/no/products/detail/kemet/C0805C105J4REC7800/8643700" (id 4) (at 198.12 153.67 0)
       (effects (font (size 1.27 1.27)) hide)
     )
@@
       (effects (font (size 1.27 1.27)) hide)
     )
-    (property "Purchase" "" (id 4) (at 205.105 96.52 0)
-      (effects (font (size 1.27 1.27)) hide)
-    )
-    (property "Order Page" "https://no.mouser.com/ProductDetail/YAGEO/RC0805FR-1310KL?qs=sGAEpiMZZMtlubZbdhIBIHucEnbnlIRRGobQQ23C9vc%3D" (id 5) (at 205.105 96.52 0)
+    (property "Purchase" "https://www.digikey.no/no/products/detail/yageo/AC0805FR-0710KL/2827834" (id 4) (at 205.105 96.52 0)
       (effects (font (size 1.27 1.27)) hide)
     )
@@
       (effects (font (size 1.27 1.27)) hide)
     )
-    (property "Purchase" "" (id 4) (at 192.405 48.895 0)
-      (effects (font (size 1.27 1.27)) hide)
-    )
-    (property "Order Page" "https://no.mouser.com/ProductDetail/Walsin/0805X105K100CT?qs=sGAEpiMZZMsh%252B1woXyUXj6GIMbU2VNPkBXHihtGsekQ%3D" (id 5) (at 192.405 48.895 0)
+    (property "Purchase" "https://www.digikey.no/no/products/detail/kemet/C0805C105J4REC7800/8643700" (id 4) (at 192.405 48.895 0)
       (effects (font (size 1.27 1.27)) hide)
     )
@@
       (effects (font (size 1.27 1.27)) hide)
     )
-    (property "Purchase" "" (id 4) (at 203.2 48.895 0)
-      (effects (font (size 1.27 1.27)) hide)
-    )
-    (property "Order Page" "https://no.mouser.com/ProductDetail/YAGEO/RC0805FR-1310KL?qs=sGAEpiMZZMtlubZbdhIBIHucEnbnlIRRGobQQ23C9vc%3D" (id 5) (at 203.2 48.895 0)
-      (effects (font (size 1.27 1.27)) hide)
-    )
+    (property "Purchase" "https://www.digikey.no/no/products/detail/yageo/AC0805FR-07100KL/5896520" (id 4) (at 203.2 48.895 0)
+      (effects (font (size 1.27 1.27)) hide)
+    )
