File: centrifuge_combined/mcu_part/power_circuit.kicad_sch (KiCad schematic)
At the start: 66 parts, among them J509 USB_B_Micro, J510 Barrel_Jack, J511 PowerIn, J512 PowerPads, Q501 Q_PMOS_DGS, U503 TPS54294, U504 TPS54294, U505 TPS54294

Commit message: make final shopping list, added to Mouser and DigiKey lists. Also budget. Swaps out TVS diodes
Parts:
- U503, U504, U505: footprint centrifuge_mcu:TSSOP-16-1EP_4.4x5mm_P0.65mm_EP3x3mm_ThermalVias_EXTRA -> Package_SO:HTSSOP-16-1EP_4.4x5mm_P0.65mm_EP3x3mm
Changed lines of the file:
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@@
     (pin "2")
   )
-  (symbol (lib_name "TPS54294_2") (lib_id "mcu_centrifuge_library:TPS54294") (at 186.055 87.63 0) (unit 1)
+  (symbol (lib_id "mcu_centrifuge_library:TPS54294") (at 186.055 87.63 0) (unit 1)
     (in_bom yes) (on_board yes)
     (property "Reference" "U504" (id 0) (at 179.705 74.93 0))
     (property "Value" "TPS54294" (id 1) (at 189.23 74.93 0))
-    (property "Footprint" "centrifuge_mcu:TSSOP-16-1EP_4.4x5mm_P0.65mm_EP3x3mm_ThermalVias_EXTRA" (id 2) (at 188.595 96.52 0)
+    (property "Footprint" "Package_SO:HTSSOP-16-1EP_4.4x5mm_P0.65mm_EP3x3mm" (id 2) (at 188.595 113.03 0)
       (effects (font (size 1.27 1.27)) hide)
     )
@@
     (property "Reference" "U505" (id 0) (at 179.705 127 0))
     (property "Value" "TPS54294" (id 1) (at 189.23 127 0))
-    (property "Footprint" "centrifuge_mcu:TSSOP-16-1EP_4.4x5mm_P0.65mm_EP3x3mm_ThermalVias_EXTRA" (id 2) (at 188.595 148.59 0)
+    (property "Footprint" "Package_SO:HTSSOP-16-1EP_4.4x5mm_P0.65mm_EP3x3mm" (id 2) (at 188.595 165.1 0)
       (effects (font (size 1.27 1.27)) hide)
     )
@@
     (pin "1")
   )
-  (symbol (lib_name "TPS54294_1") (lib_id "mcu_centrifuge_library:TPS54294") (at 186.055 34.29 0) (unit 1)
+  (symbol (lib_id "mcu_centrifuge_library:TPS54294") (at 186.055 34.29 0) (unit 1)
     (in_bom yes) (on_board yes)
     (property "Reference" "U503" (id 0) (at 179.705 21.59 0))
     (property "Value" "TPS54294" (id 1) (at 189.23 21.59 0))
-    (property "Footprint" "centrifuge_mcu:TSSOP-16-1EP_4.4x5mm_P0.65mm_EP3x3mm_ThermalVias_EXTRA" (id 2) (at 188.595 59.69 0)
-      (effects (font (size 1.27 1.27)) hide)
-    )
+    (property "Footprint" "Package_SO:HTSSOP-16-1EP_4.4x5mm_P0.65mm_EP3x3mm" (id 2) (at 188.595 59.69 0)
+      (effects (font (size 1.27 1.27)) hide)
+    )
