File: centrifuge_combined/fpga_part/config_sram.kicad_sch (KiCad schematic)
At the start: 5 parts, among them U1 XC7A100T-FTG256, U2 S25FL127SABMFV10, U3 CY7C1370KV33

Commit message: fix JTAG Vref, pullup on CS and remove SRAM_CS1p3
Parts:
- added R55: 2.2k, Resistor_SMD:R_0805_2012Metric_Pad1.20x1.40mm_HandSolder, symbol Device:R_Small
Connections:
- net +3V3_FPGA: now also R55.2
- net GND: now also U3.92 (~{CE3}), U3.98 (~{CE1})
- net n_CONFIG_CS: now also R55.1
- removed net SRAM_CE1: U1.P8 (IO_L20P_T3_A08_D24_14), U3.92 (~{CE3}), U3.98 (~{CE1})
- no-connect marks 20 -> 21
Other:
- note added: "UG470 pg 51 shows these pullups, as does lecture (2.4k instead of 2.2k)"
- note removed: "Tying these together because separate CEs would be for multiple accessors"
Changed lines of the file:
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@@
   (junction (at 168.275 20.32) (diameter 0) (color 0 0 0 0)
   )
+  (junction (at 48.26 19.685) (diameter 0) (color 0 0 0 0)
+  )
   (junction (at 164.465 88.9) (diameter 0) (color 0 0 0 0)
   )
@@
   (junction (at 280.67 155.575) (diameter 0) (color 0 0 0 0)
   )
+  (junction (at 221.615 22.225) (diameter 0) (color 0 0 0 0)
+  )
   (junction (at 164.465 111.76) (diameter 0) (color 0 0 0 0)
   )
@@
   (junction (at 66.675 43.815) (diameter 0) (color 0 0 0 0)
   )
+  (junction (at 31.75 31.115) (diameter 0) (color 0 0 0 0)
+  )
   (junction (at 64.135 43.815) (diameter 0) (color 0 0 0 0)
   )
@@
   )
   (junction (at 224.155 155.575) (diameter 0) (color 0 0 0 0)
+  )
+  (junction (at 226.695 22.225) (diameter 0) (color 0 0 0 0)
   )
   (junction (at 71.755 43.815) (diameter 0) (color 0 0 0 0)
@@
   (no_connect (at 48.895 160.655))
   (no_connect (at 48.895 130.175))
+  (no_connect (at 48.895 163.195))
   (no_connect (at 150.495 94.615))
   (no_connect (at 150.495 92.075))
@@
     (stroke (width 0) (type default) (color 0 0 0 0))
   )
+  (wire (pts (xy 29.845 31.115) (xy 31.75 31.115))
+    (stroke (width 0) (type default) (color 0 0 0 0))
+  )
   (wire (pts (xy 226.695 134.62) (xy 226.695 152.4))
     (stroke (width 0) (type default) (color 0 0 0 0))
@@
     (stroke (width 0) (type default) (color 0 0 0 0))
   )
+  (wire (pts (xy 31.75 19.685) (xy 31.75 22.86))
+    (stroke (width 0) (type default) (color 0 0 0 0))
+  )
+  (wire (pts (xy 221.615 35.56) (xy 221.615 22.225))
+    (stroke (width 0) (type default) (color 0 0 0 0))
+  )
   (wire (pts (xy 61.595 43.815) (xy 64.135 43.815))
     (stroke (width 0) (type default) (color 0 0 0 0))
@@
     (stroke (width 0) (type default) (color 0 0 0 0))
   )
-  (wire (pts (xy 117.475 28.575) (xy 120.015 28.575))
+  (wire (pts (xy 69.215 19.685) (xy 48.26 19.685))
     (stroke (width 0) (type default) (color 0 0 0 0))
   )
@@
     (stroke (width 0) (type default) (color 0 0 0 0))
   )
+  (wire (pts (xy 31.75 27.94) (xy 31.75 31.115))
+    (stroke (width 0) (type default) (color 0 0 0 0))
+  )
   (wire (pts (xy 59.055 43.815) (xy 61.595 43.815))
     (stroke (width 0) (type default) (color 0 0 0 0))
@@
     (stroke (width 0) (type default) (color 0 0 0 0))
   )
+  (wire (pts (xy 221.615 22.225) (xy 206.375 22.225))
+    (stroke (width 0) (type default) (color 0 0 0 0))
+  )
   (wire (pts (xy 104.775 22.225) (xy 104.775 31.75))
     (stroke (width 0) (type default) (color 0 0 0 0))
@@
     (stroke (width 0) (type default) (color 0 0 0 0))
   )
+  (wire (pts (xy 48.26 19.685) (xy 48.26 23.495))
+    (stroke (width 0) (type default) (color 0 0 0 0))
+  )
   (wire (pts (xy 219.075 158.115) (xy 220.345 158.115))
     (stroke (width 0) (type default) (color 0 0 0 0))
@@
     (stroke (width 0) (type default) (color 0 0 0 0))
   )
+  (wire (pts (xy 31.75 31.115) (xy 33.02 31.115))
+    (stroke (width 0) (type default) (color 0 0 0 0))
+  )
   (wire (pts (xy 127.635 43.815) (xy 130.175 43.815))
     (stroke (width 0) (type default) (color 0 0 0 0))
@@
     (stroke (width 0) (type default) (color 0 0 0 0))
   )
+  (wire (pts (xy 48.26 19.685) (xy 31.75 19.685))
+    (stroke (width 0) (type default) (color 0 0 0 0))
+  )
   (wire (pts (xy 226.695 22.225) (xy 280.67 22.225))
     (stroke (width 0) (type default) (color 0 0 0 0))
@@
     (stroke (width 0) (type default) (color 0 0 0 0))
   )
+  (wire (pts (xy 221.615 22.225) (xy 226.695 22.225))
+    (stroke (width 0) (type default) (color 0 0 0 0))
+  )
   (wire (pts (xy 63.5 31.115) (xy 88.9 31.115))
     (stroke (width 0) (type default) (color 0 0 0 0))
   )
+  (wire (pts (xy 206.375 22.225) (xy 206.375 35.56))
+    (stroke (width 0) (type default) (color 0 0 0 0))
+  )
   (wire (pts (xy 283.21 86.36) (xy 283.21 96.52))
     (stroke (width 0) (type default) (color 0 0 0 0))
@@
     (stroke (width 0) (type default) (color 0 0 0 0))
   )
-  (wire (pts (xy 117.475 28.575) (xy 117.475 31.115))
-    (stroke (width 0) (type default) (color 0 0 0 0))
-  )
   (wire (pts (xy 283.21 73.66) (xy 283.21 86.36))
     (stroke (width 0) (type default) (color 0 0 0 0))
@@
     (stroke (width 0) (type default) (color 0 0 0 0))
   )
-  (text "Tying these together because separate CEs\nwould be for multiple accessors"
-    (at 107.315 24.765 0)
-    (effects (font (size 1.27 1.27)) (justify left bottom))
-  )
   (text "Don't bother with sleep mode" (at 222.885 161.29 0)
     (effects (font (size 1.27 1.27)) (justify left bottom))
@@
   )
   (text "IO2/3 pull ups from XAPP586 pg7\nNeither this nor flash datasheets\nmention pullup/open-drain but\nincluding footprints just in case."
-    (at 46.355 20.955 0)
-    (effects (font (size 1.27 1.27)) (justify right bottom))
+    (at 44.45 8.89 180)
+    (effects (font (size 1.27 1.27)) (justify right bottom))
+  )
+  (text "UG470 pg 51 shows these pullups, as does lecture\n(2.4k instead of 2.2k)\n"
+    (at 15.875 18.415 0)
+    (effects (font (size 1.27 1.27)) (justify left bottom))
   )
   (text "All I/O on the SRAM is 3.3 V,\nbut it can run at 2.5 V apparently"
@@
     (effects (font (size 1.27 1.27)) (justify right bottom))
   )
-  (label "SRAM_CE3" (at 221.615 35.56 90)
-    (effects (font (size 1.27 1.27)) (justify left bottom))
-  )
-  (label "SRAM_CE3" (at 117.475 31.115 180)
-    (effects (font (size 1.27 1.27)) (justify right bottom))
-  )
   (label "SRAM_MODE" (at 184.15 158.115 180)
     (effects (font (size 1.27 1.27)) (justify right bottom))
@@
     (effects (font (size 1.27 1.27)) (justify left bottom))
   )
-  (label "SRAM_CE1p3" (at 48.895 163.195 180)
-    (effects (font (size 1.27 1.27)) (justify right bottom))
-  )
   (label "SRAM_ADV_LD" (at 48.895 142.875 180)
     (effects (font (size 1.27 1.27)) (justify right bottom))
@@
     (effects (font (size 1.27 1.27)) (justify left bottom))
   )
-  (label "SRAM_CE1" (at 117.475 28.575 180)
-    (effects (font (size 1.27 1.27)) (justify right bottom))
-  )
   (label "SRAM_D12" (at 150.495 130.175 0)
     (effects (font (size 1.27 1.27)) (justify left bottom))
@@
     (effects (font (size 1.27 1.27)) (justify left bottom))
   )
-  (label "SRAM_CE1" (at 206.375 35.56 90)
-    (effects (font (size 1.27 1.27)) (justify left bottom))
-  )
   (label "SRAM_D3" (at 150.495 153.035 0)
     (effects (font (size 1.27 1.27)) (justify left bottom))
@@
     (effects (font (size 1.27 1.27)) (justify left bottom))
   )
-  (label "SRAM_CE1p3" (at 120.015 28.575 0)
-    (effects (font (size 1.27 1.27)) (justify left bottom))
-  )
   (label "SRAM_A2" (at 211.455 134.62 270)
     (effects (font (size 1.27 1.27)) (justify right bottom))
@@
     (effects (font (size 1.27 1.27)) (justify left bottom))
   )
-  (label "n_CONFIG_CS" (at 33.02 31.115 180)
+  (label "n_CONFIG_CS" (at 29.845 31.115 180)
     (effects (font (size 1.27 1.27)) (justify right bottom))
   )
@@
     )
     (pin "1")
+  )
+  (symbol (lib_id "Device:R_Small") (at 31.75 25.4 180) (unit 1)
+    (in_bom yes) (on_board yes)
+    (property "Reference" "R55" (id 0) (at 26.67 24.13 0)
+      (effects (font (size 1.27 1.27)) (justify right))
+    )
+    (property "Value" "2.2k" (id 1) (at 26.035 26.035 0)
+      (effects (font (size 1.27 1.27)) (justify right))
+    )
+    (property "Footprint" "Resistor_SMD:R_0805_2012Metric_Pad1.20x1.40mm_HandSolder" (id 2) (at 31.75 25.4 0)
+      (effects (font (size 1.27 1.27)) hide)
+    )
+    (property "Datasheet" "~" (id 3) (at 31.75 25.4 0)
+      (effects (font (size 1.27 1.27)) hide)
+    )
+    (property "Purchase" "" (id 4) (at 31.75 25.4 0)
+      (effects (font (size 1.27 1.27)) hide)
+    )
+    (property "Order Page" "https://no.mouser.com/ProductDetail/Vishay-Dale/CRCW08052K20FKEB?qs=sGAEpiMZZMtlubZbdhIBINvvmcV35a3LmL3hFYkil7g%3D" (id 5) (at 31.75 25.4 0)
+      (effects (font (size 1.27 1.27)) hide)
+    )
+    (pin "1")
+    (pin "2")
   )
   (symbol (lib_id "power:GND") (at 220.345 159.385 0) (unit 1)
@@
     (pin "2")
   )
-  (symbol (lib_id "centrifuge_symbols:+3V3_FPGA") (at 48.26 23.495 0) (unit 1)
-    (in_bom yes) (on_board yes) (fields_autoplaced)
-    (property "Reference" "#PWR0215" (id 0) (at 48.26 27.305 0)
-      (effects (font (size 1.27 1.27)) hide)
-    )
-    (property "Value" "+3V3_FPGA" (id 1) (at 48.26 19.939 90)
-      (effects (font (size 1.27 1.27)) (justify left))
-    )
-    (property "Footprint" "" (id 2) (at 48.26 23.495 0)
-      (effects (font (size 1.27 1.27)) hide)
-    )
-    (property "Datasheet" "" (id 3) (at 48.26 23.495 0)
-      (effects (font (size 1.27 1.27)) hide)
-    )
-    (pin "1")
-  )
   (symbol (lib_id "centrifuge_symbols:S25FL127SABMFV10") (at 48.26 33.655 0) (unit 1)

Commit message: make final shopping list, added to Mouser and DigiKey lists. Also budget. Swaps out TVS diodes
Parts:
- U2: Order Page https://www.digikey.no/en/products/detail/winbond-electroni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 -> https://www.digikey.no/en/products/detail/cypress-semicondu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
Changed lines of the file:
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@@
       (effects (font (size 1.27 1.27)) hide)
     )
-    (property "Datasheet" "https://www.winbond.com/resource-files/w25q64jv%20revj%2003272018%20plus.pdf" (id 3) (at 48.26 33.655 0)
+    (property "Datasheet" "https://www.infineon.com/dgdl/Infineon-S25FL127S_128-Mb_(16_MB)_3.0_V_SPI_Flash_Memory-DataSheet-v11_00-EN.pdf?fileId=8ac78c8c7d0d8da4017d0ecfa58c49f7&utm_source=cypress&utm_medium=referral&utm_campaign=202110_globe_en_all_integration-files" (id 3) (at 48.26 33.655 0)
       (effects (font (size 1.27 1.27)) hide)
     )
-    (property "Order Page" "https://www.digikey.no/en/products/detail/winbond-electronics/W25Q64JVSSIQ/5803992" (id 4) (at 48.26 33.655 0)
+    (property "Order Page" "https://www.digikey.no/en/products/detail/cypress-semiconductor-corp/S25FL127SABMFV101/5788556" (id 4) (at 48.26 33.655 0)
       (effects (font (size 1.27 1.27)) hide)
     )
