File: centrifuge_combined/fpga_part/vga_interface.kicad_sch (KiCad schematic)
At the start: 19 parts, among them J3 Conn_01x15, Q3 BSN20, Q4 BSN20, U13 RCLAMP0524PATCT, U9 LSF0102

Commit message: fix duplicate Cs, add extra ACD/DAC and breakout, and fix TVS schematic hidden pin
Parts:
- U13: Order Page https://no.mouser.com/ProductDetail/Semtech/RCLAMP0524PATCT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 -> https://www.digikey.no/en/products/detail/diodes-incorporat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
Connections:
- net GND: now also U13.3 (GND)
Changed lines of the file:
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@@
       (effects (font (size 1.27 1.27)) hide)
     )
-    (property "Datasheet" "https://no.mouser.com/datasheet/2/761/SEMT_S_A0005071119_1-2575775.pdf" (id 3) (at 213.868 115.062 0)
+    (property "Datasheet" "https://www.diodes.com/assets/Datasheets/D5V0FS4U10LP.pdf" (id 3) (at 213.868 115.062 0)
       (effects (font (size 1.27 1.27)) hide)
     )
-    (property "Order Page" "https://no.mouser.com/ProductDetail/Semtech/RCLAMP0524PATCT?qs=rBWM4%252BvDhIcnc1nesEh7XA%3D%3D" (id 4) (at 213.868 115.062 0)
+    (property "Order Page" "https://www.digikey.no/en/products/detail/diodes-incorporated/D5V0FS4U10LP-7/7930773" (id 4) (at 213.868 115.062 0)
       (effects (font (size 1.27 1.27)) hide)
     )
