File: centrifuge_combined/fpga_part/vga_input.kicad_sch (KiCad schematic)
At the start: 45 parts, among them U4 TVP7002, X1 ECS-2333-270-BN

Commit message: change resistor values to have to 2k2, and also make I2C hopefully work
Parts:
- R23, R24: value 2.2k -> DNI
- R25, R26: value 2.2k -> 4.7k
Other:
- note added: "Used to be 2.2k"
- note added: "Used to be 2.2k Connect only one of them 3V3 on adc2, GND on adc1"
Changed lines of the file:
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@@
     (stroke (width 0) (type default) (color 0 0 0 0))
+  )
+  (text "Used to be 2.2k" (at 231.902 67.31 0)
+    (effects (font (size 1.27 1.27)) (justify left bottom))
+  )
+  (text "Used to be 2.2k\nConnect only one of them\n3V3 on adc2, GND on adc1"
+    (at 275.082 69.85 0)
+    (effects (font (size 1.27 1.27)) (justify left bottom))
   )
   (text "This one is supposed to be a separate rail." (at 106.68 172.72 0)
@@
   (symbol (lib_id "Device:R_Small") (at 241.935 63.5 0) (unit 1)
     (in_bom yes) (on_board yes) (fields_autoplaced)
-    (property "Reference" "R24" (id 0) (at 244.475 62.2299 0)
-      (effects (font (size 1.27 1.27)) (justify left))
-    )
-    (property "Value" "2.2k" (id 1) (at 244.475 64.7699 0)
+    (property "Reference" "R24" (id 0) (at 243.84 62.2299 0)
+      (effects (font (size 1.27 1.27)) (justify left))
+    )
+    (property "Value" "DNI" (id 1) (at 243.84 64.7699 0)
       (effects (font (size 1.27 1.27)) (justify left))
     )
@@
       (effects (font (size 1.27 1.27)) (justify left))
     )
-    (property "Value" "2.2k" (id 1) (at 269.24 82.5499 0)
+    (property "Value" "4.7k" (id 1) (at 269.24 82.5499 0)
       (effects (font (size 1.27 1.27)) (justify left))
     )
@@
       (effects (font (size 1.27 1.27)) (justify left))
     )
-    (property "Value" "2.2k" (id 1) (at 236.22 64.7699 0)
+    (property "Value" "DNI" (id 1) (at 236.22 64.7699 0)
       (effects (font (size 1.27 1.27)) (justify left))
     )
@@
       (effects (font (size 1.27 1.27)) (justify left))
     )
-    (property "Value" "2.2k" (id 1) (at 269.24 64.7699 0)
-      (effects (font (size 1.27 1.27)) (justify left))
-    )
+    (property "Value" "4.7k" (id 1) (at 269.24 64.7699 0)
+      (effects (font (size 1.27 1.27)) (justify left))
+    )
