File: centrifuge_combined/fpga_part/vga_output.kicad_sch (KiCad schematic)
At the start: 15 parts, among them U5 THS8136

Commit message: change resistor values to have to 2k2, and also make I2C hopefully work
Parts:
- R7: value 2.2k -> 4.7k
Other:
- note added: "Used to be 2.2k"
Changed lines of the file:
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@@
     (stroke (width 0) (type default) (color 0 0 0 0))
+  )
+  (text "Used to be 2.2k" (at 239.014 143.256 0)
+    (effects (font (size 1.27 1.27)) (justify left bottom))
   )
   (text "datasheet recommends 3.8k on rfsadj\nfor our 700 mV outputs"
@@
       (effects (font (size 1.27 1.27)) (justify left))
     )
-    (property "Value" "2.2k" (id 1) (at 236.22 144.7799 0)
-      (effects (font (size 1.27 1.27)) (justify left))
-    )
+    (property "Value" "4.7k" (id 1) (at 236.22 144.7799 0)
+      (effects (font (size 1.27 1.27)) (justify left))
+    )
