File: centrifuge_combined/fpga_part/fpga_part.kicad_sch (KiCad schematic)
At the start: 8 parts, among them X3 EC2620TTS-100.000MTR

Commit message: change resistor values to have to 2k2, and also make I2C hopefully work
Changed lines of the file:
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@@
     (effects (font (size 1.27 1.27)) (justify right bottom))
   )
-  (label "SDA_MCU_SL0" (at 66.675 41.91 0)
+  (label "SDA_MCU_SL2" (at 66.675 41.91 0)
     (effects (font (size 1.27 1.27)) (justify left bottom))
   )
@@
     (effects (font (size 1.27 1.27)) (justify right bottom))
   )
-  (label "SCL_MCU_SL0" (at 66.675 43.815 0)
+  (label "SCL_MCU_SL2" (at 66.675 43.815 0)
     (effects (font (size 1.27 1.27)) (justify left bottom))
   )
@@
     (effects (font (size 1.27 1.27)) (justify left bottom))
   )
-  (label "SCL_MCU_SL0" (at 248.031 78.105 180)
+  (label "SCL_MCU_SL1" (at 248.031 78.105 180)
     (effects (font (size 1.27 1.27)) (justify right bottom))
   )
@@
     (effects (font (size 1.27 1.27)) (justify right bottom))
   )
-  (label "SDA_MCU_SL0" (at 248.031 80.645 180)
+  (label "SDA_MCU_SL1" (at 248.031 80.645 180)
     (effects (font (size 1.27 1.27)) (justify right bottom))
   )
@@
     (effects (font (size 1.27 1.27)) (justify left bottom))
   )
-  (label "SCL_MCU_SL1" (at 248.031 93.345 180)
+  (label "SCL_MCU_SL2" (at 248.031 93.345 180)
     (effects (font (size 1.27 1.27)) (justify right bottom))
   )
@@
     (effects (font (size 1.27 1.27)) (justify right bottom))
   )
-  (label "SDA_MCU_SL1" (at 248.031 95.885 180)
+  (label "SDA_MCU_SL2" (at 248.031 95.885 180)
     (effects (font (size 1.27 1.27)) (justify right bottom))
   )
@@
     (effects (font (size 1.27 1.27)) (justify left))
   )
-  (hierarchical_label "SCL_MCU_SL0" (shape input) (at 251.587 78.105 0)
+  (hierarchical_label "SCL_MCU_SL1" (shape input) (at 251.587 78.105 0)
     (effects (font (size 1.27 1.27)) (justify left))
   )
@@
     (effects (font (size 1.27 1.27)) (justify left))
   )
-  (hierarchical_label "SDA_MCU_SL0" (shape input) (at 251.587 80.645 0)
+  (hierarchical_label "SDA_MCU_SL1" (shape input) (at 251.587 80.645 0)
     (effects (font (size 1.27 1.27)) (justify left))
   )
@@
     (effects (font (size 1.27 1.27)) (justify left))
   )
-  (hierarchical_label "SDA_MCU_SL1" (shape input) (at 251.587 95.885 0)
+  (hierarchical_label "SDA_MCU_SL2" (shape input) (at 251.587 95.885 0)
     (effects (font (size 1.27 1.27)) (justify left))
   )
@@
     (effects (font (size 1.27 1.27)) (justify left))
   )
-  (hierarchical_label "SCL_MCU_SL1" (shape input) (at 251.587 93.345 0)
+  (hierarchical_label "SCL_MCU_SL2" (shape input) (at 251.587 93.345 0)
     (effects (font (size 1.27 1.27)) (justify left))
   )

Commit message: change the names of some named wires in the schematic, to make numbering more consistent
Changed lines of the file:
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@@
     (effects (font (size 1.27 1.27)) (justify right bottom))
   )
-  (label "MCU_ADC0_RST" (at 248.031 83.185 180)
+  (label "MCU_ADC2_RST" (at 248.031 83.185 180)
     (effects (font (size 1.27 1.27)) (justify right bottom))
   )
@@
     (effects (font (size 1.27 1.27)) (justify right bottom))
   )
-  (label "MCU_ADC0_RST" (at 95.25 41.91 180)
+  (label "MCU_ADC2_RST" (at 95.25 41.91 180)
     (effects (font (size 1.27 1.27)) (justify right bottom))
   )
@@
     (effects (font (size 1.27 1.27)) (justify left))
   )
-  (hierarchical_label "MCU_ADC0_RST" (shape input) (at 251.587 83.185 0)
+  (hierarchical_label "MCU_ADC2_RST" (shape input) (at 251.587 83.185 0)
     (effects (font (size 1.27 1.27)) (justify left))
   )

Commit message: fix mismatch between VSYNC and HSYNC out, only needs a swap in constraints file as well
Changed lines of the file:
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@@
       (effects (font (size 1.27 1.27)) (justify left top))
     )
-    (pin "VSYNC_OUT0" output (at 176.403 42.291 0)
+    (pin "HSYNC_OUT0" output (at 176.403 42.291 0)
       (effects (font (size 1.27 1.27)) (justify right))
     )
-    (pin "HSYNC_OUT0" output (at 176.403 44.196 0)
+    (pin "VSYNC_OUT0" output (at 176.403 44.196 0)
       (effects (font (size 1.27 1.27)) (justify right))
     )
