File: centrifuge_combined/fpga_part/ddc_eeprom.kicad_sch (KiCad schematic)
At the start: 9 parts, among them U10 M24C02-WMN

Commit message: fully commit to calling top VGA ADC2
Other:
- note added: "Writes are enabled if pulled to GND or left floating"
Changed lines of the file:
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@@
     (stroke (width 0) (type default) (color 0 0 0 0))
+  )
+  (text "Writes are enabled if pulled to GND or left floating"
+    (at 163.83 106.172 0)
+    (effects (font (size 1.27 1.27)) (justify left bottom))
   )
   (label "SDA" (at 209.55 113.665 270)
